Commit message: fix(urdf): 把 LIO 的 body 帧挂到 imu_link 下，修 cartographer use_odometry 建图停摆
确证链（都在本仓源码里）：
1) use_odometry=true -> cartographer 订阅 /odom（FAST-LIO 的），其 child_frame_id="body"
   （FAST_LIO/src/laserMapping.cpp:631）
2) SensorBridge::ToOdometryData（sensor_bridge.cpp:51-62）里 LookupToTracking(time,"body")
   -> tf_bridge.cpp:53 查 TF imu_link<-body 失败（用户实跑日志 10Hz 刷
      "Could not find a connection between 'imu_link' and 'body' because they are not
       part of the same tree"）-> 返回 nullptr
3) HandleOdometryMessage（sensor_bridge.cpp:66-70）里 if(odometry_data != nullptr) 不成立
   -> 该条 odom 什么都不做 -> OrderedMultiQueue 一直等 odom 传感器 -> **建图停摆**
   （这就是"开了 use_odometry 反而无法建图"的原因）

修复：body 就是 IMU 那一帧（FAST-LIO 的 extrinsic_T=[0,0,0.05] -> IMU 在雷达下方 5cm
= URDF 的 imu_link），所以在 sentry_robot_sim.xacro 里显式加
  link "body" + fixed joint imu_link->body（恒等）
由 robot_state_publisher 以静态 TF 发布。比在 launch 里另起 static_transform_publisher
更稳：不依赖启动条件、不受 lio/mode 组合影响。

撤销上一版 launch 里的 tf_body_alias_node（已由 URDF 承担）。

验证：xacro 展开 OK（含 body link 与 body_alias_joint，identity）；install 侧 xacro 是软链
（不用 rebuild）；launch 解析 25 actions。

已知交互（待处理）：mode:=nav 且 localization:=''（T1 回退用法）下，URDF 的
imu_link->body 与 T1 的 body->odom 会形成 TF 环；T3 之后 lio_tf_adapter 已提供
odom->base_link，最干净的做法是删掉 T1 的 body->odom。mapping/slam_nav/nav+具体重定位
不受影响。

File: src/rm_nav_bringup/urdf/sentry_robot_sim.xacro (robot description, xacro)
@@ -166,4 +166,19 @@
     </inertial>
   </link>
+  <!-- body：FAST-LIO / Point-LIO 里程计消息里的 child_frame_id（就是 IMU 帧本身）。
+       ★ 2026-09-21：显式把它挂到 imu_link 下（恒等），否则 cartographer 的 use_odometry
+       在 SensorBridge::ToOdometryData 里查 TF `imu_link ← body` 会失败
+       （tf_bridge.cpp:53 "Tf has two or more unconnected trees"）→ 该条 odom 被整个丢弃
+       → 轨迹构建器的 collator 一直等 odom 传感器 → **建图停摆**。
+       恒等是正确的：FAST-LIO 的 extrinsic_T=[0,0,0.05] 表示 IMU 就在雷达下方 5cm，
+       即 URDF 的 imu_link，所以 body ≡ imu_link。 -->
+  <link name="body">
+    <xacro:default_inertial mass="1e-6"/>
+  </link>
+  <joint name="body_alias_joint" type="fixed">
+    <parent link="imu_link"/>
+    <child link="body"/>
+    <origin xyz="0 0 0" rpy="0 0 0"/>
+  </joint>
   <!-- Gazebo插件设置相关 -->
   <gazebo reference="base_link">

Commit message: fix(lio): odom 的 child_frame_id 由 body 改为 imu_link，修 cartographer use_odometry 连不上 TF
上一版把 body 挂到 URDF 的 imu_link 下是错的：FAST-LIO 自己也在广播 TF
camera_init->body（laserMapping.cpp:649），于是 body 有两个父帧 -> tf2 里 body 实际
挂在 LIO 那棵树（camera_init）下，而 camera_init 与机器人树毫无连接 ->
cartographer 查 imu_link<-body 仍然失败（用户日志：robot_state_publisher 已
"got segment body"，但 tf_bridge.cpp:53 仍刷 "two or more unconnected trees"）。

正确改法：让 odom 消息的 child_frame_id 直接就是 imu_link —— 它本来就是 IMU 的位姿
（FAST-LIO 的 extrinsic_T=[0,0,0.05] 说明 IMU 在雷达下方 5cm = URDF imu_link），
语义完全正确；cartographer 的 LookupToTracking(imu_link, imu_link) 得到恒等变换。
- src/rm_localization/FAST_LIO/src/laserMapping.cpp:631  body -> imu_link
- src/rm_localization/point_lio/src/laserMapping.cpp:246  body -> imu_link
- 撤回 sentry_robot_sim.xacro 里的 body link/joint（避免双父）

lio_tf_adapter 只读 odom 的 pose（不读 child_frame_id），且靠自己的 xyz 杆臂补偿，
所以不受影响。

⚠️ 改了 C++ 源码 -> 需要重新 build（正在跑 colcon build --packages-select fast_lio point_lio）。

File: src/rm_nav_bringup/urdf/sentry_robot_sim.xacro (robot description, xacro)
@@ -166,19 +166,4 @@
     </inertial>
   </link>
-  <!-- body：FAST-LIO / Point-LIO 里程计消息里的 child_frame_id（就是 IMU 帧本身）。
-       ★ 2026-09-21：显式把它挂到 imu_link 下（恒等），否则 cartographer 的 use_odometry
-       在 SensorBridge::ToOdometryData 里查 TF `imu_link ← body` 会失败
-       （tf_bridge.cpp:53 "Tf has two or more unconnected trees"）→ 该条 odom 被整个丢弃
-       → 轨迹构建器的 collator 一直等 odom 传感器 → **建图停摆**。
-       恒等是正确的：FAST-LIO 的 extrinsic_T=[0,0,0.05] 表示 IMU 就在雷达下方 5cm，
-       即 URDF 的 imu_link，所以 body ≡ imu_link。 -->
-  <link name="body">
-    <xacro:default_inertial mass="1e-6"/>
-  </link>
-  <joint name="body_alias_joint" type="fixed">
-    <parent link="imu_link"/>
-    <child link="body"/>
-    <origin xyz="0 0 0" rpy="0 0 0"/>
-  </joint>
   <!-- Gazebo插件设置相关 -->
   <gazebo reference="base_link">
