Commit message: feat(robot11): Phase 3 —— 让雷达真的看得见（A 方案：碰撞挖视锥）+ 斜置感知链槽位化 + nav2 几何覆盖
用户判定（2026-10-07）：30° 是绕 **roll**（按实物确认）；上游 URDF/mesh 仿真侧可改（每处偏离登记）。

Phase 2 的"75.5% 自击 / 地面 529 点每帧 / 无 /odom"是**三个根因叠在一起**，本轮全部定位：
 ① `body` 的 4 个 DP box 是实心包络，而雷达原点 z=0.157 落在第 4 个 box（顶 0.213）**内部**
    ⇒ 离线 30000 条同源射线实测 **80.5% 落在 <0.12 m**、看见地面 0%；
 ② 模型根 link 叫 `body`，而全链路契约帧名是 `base_link`（small_point_lio 源码硬编码 lookup）
    ⇒ **TF 断成两棵树**、`/odom` 0 条；上游自己的 SolidWorks CSV 里这个 link 本来就叫 base_link
    ⇒ 生成时改名；
 ③ linefit 的 gravity_aligned_frame 路径曾因 Eigen 未初始化把点云塌到原点（已单独修）。
显式排除：④ C（抽稀网格碰撞）——spawn 服务 60 s 超时，但日志证明**插件已挂上并初始化**，
    根因是 ODE 的 ray-vs-trimesh 是 O(三角面数)（30000×3000 ≈ 9e7 次/帧）⇒ 路径不可用，非参数问题。

A 方案（**采用**）：`body` 碰撞 = 4 个 DP box **减去雷达视锥**（锥半角 100.22°、半径 0.5 m、
内清空 0.05 m、体素 15 mm、保守角点判定）后分解成 **76 个 box**；生成器新增 `--body-collision carved`
（另有 boxes / mesh 供对照），清单落 `robot11_description/inventory/livox_fov_boxes.json`（含验证数字）。
B 方案（抬高雷达）实现为 `--livox-raise-m` + launch `livox_raise_m`（默认 0 = 上游几何），
离线扫描：+0.05 m 仍 96.6% 自击、**+0.08 m 才干净**、+0.10 m 起与 A 等价 ⇒ 不采用（几何偏离更大）。
云台 l10/l11 的碰撞由"单个包围盒"换成网格推出的 7/22 个 box（包围盒离雷达只有 0.099/0.091 m 且实心，
实测 34.7% 的射线打在它面上；真网格最近 0.116/0.139 m）。

斜置感知链（**只对本槽位生效**）：
 · `livox_frame` 帧重力对齐（joint rpy=0），30° 倾角放进插件 `<tilt_rpy>`（射线真的斜、点云在父 link 系）
   ⇒ linefit/p2l 都不需要 gravity_aligned_frame / target_frame（顺手保住 p2l 的 target_frame="" 加固）；
 · 新增槽位配置 `linefit config/segmentation_sim_robot11.yaml`：**只改 sensor_height 0.226 → 0.2595**；
 · LIO 外参**不动**（IMU 与雷达仍是 0.05 m 纯平移 ⇒ extrinsic_T=[0,0,0.05]、R=I 逐字节成立）；
 · nav2 几何**槽位覆盖层**：新增 `rm_nav_bringup/config/nav2_params_sim_robot11_costmap.yaml`
   （robot_radius 0.3565 = 凸包外接、inflation 0.70/0.75），launch 里 `_Nav2ParamsForSlot` 深合并，
   默认/hzmirm **原样返回公共段路径**（单元级验证：0.22/0.5/0.55 不变）；
 · `spin_speed` 对 robot11 默认 **0.0**（轮子是真 cylinder、云台无控制器），其它槽位仍 5.0。

实测（无头隔离、RMUL2026、mode:=mapping、静止 20 s + 直行 8 s + 原地偏航 5 s）：
 · **/odom 188 条**（Phase 2 = 0）· **ground 5637 点/帧**（Phase 2 = 529；默认模型 2739）
 · **/scan >4 m ≈81 波束/帧**（Phase 2 = 0）· <1 m ≈521/帧 · 最近 0.05 m · 点数/帧 11951
 · 自击 r<0.12 = **29.0%**（Phase 2 = 75.5%；离线归因：近点 100% 是**云台**，中位 0.14 m，物理真实）
 · LIO 漂移（位移差口径）：直线 **0.024 m / 0.26°**、偏航 **0.0002 m / 0.004°**（默认模型 0.006/0.03°、0.0008/0.005°）
 · RTF 0.46（默认 0.79；代价主要来自"链路现在真的在算"）

工具：新增 `tools/scripts/regress/robot11_livox_fov.py`（离线筛方案：mesh/4box/挖视锥三选一 +
生成 A 的 box 与云台细盒 + 与 Gazebo 同源的 30000 条射线统计）；`robot_model_probe.py` 新增
`--yaw-seconds/--yaw-rate` 与 `phase_drift`（**位移差**口径，修正 Phase 2 里把"出生点偏移"当漂移的读法）、
`cloud_selfhit_frac` 精确计数、`ground_r_hist`（量 speed_limit_lookahead_m 是否有效）。

文档：docs/robot_models.md 新增 §11（A/B/C 实测、9 条偏离 provenance 表、斜置链处理与验证、
槽位配置增量、nav2 覆盖层、try/rollback、未验证清单）+ §11.4 对 §3.3 的诚实更正。
默认模型与所有默认配置逐字节未改。

File: src/rm_nav_bringup/urdf/sentry_robot_robot11_sim.xacro (robot description, xacro)
@@ -27,4 +27,28 @@
     【上游原样】= 与上游 URDF 数值逐字相同（脚本生成，可重算）
     【我们加的】= 本栈要跑起来必须补的（逐条写理由与日期）
+  ── Phase 3（2026-10-07）：让雷达"看得出去" + 斜置感知链 ─────────────────────
+    用户的判定（两条，都已按它执行）：
+      (1) **30° 是绕 roll**（用户按实物确认）⇒ 本文件的默认 `livox_tilt_rpy` = roll 形式；
+      (2) 上游 URDF/mesh "跟实物基本一致，仿真侧可以改" ⇒ 允许仿真侧适配，
+         但**每一处偏离都要写日期 + 中文理由 + provenance 表**（见 docs/robot_models.md §11）。
+    Phase 2 的结论是"这台车的雷达在底盘凹槽里，看不见外面"（75.5% 的点是自击、无 /odom）。
+    Phase 3 用**三种方案**实测（离线 30000 条射线 + Gazebo 无头跑）：
+      A（保真优先，**采用**）：body 碰撞 = DP box 减视锥（`—body-collision carved`）⇒ 雷达仍在
+         上游的 0.2595 m 高度，只把"凹槽开口"在碰撞里显式挖出来；
+      B（仿真适配）：保留 4 个 box，把 `livox_frame` 抬高（`—livox-raise-m`）⇒ 离线扫描：
+         +0.05 m 仍 96.6% 自击、+0.06 m 降到 19.8%、**+0.08 m 才干净（0.24%）**、
+         +0.10 m 起与 A 等价（0% 自击 / 25.2% 看见地面）—— 代价是雷达离地 0.2595 → 0.3595 m，
+         与本仓默认模型的 0.226 m 差得更远，且 linefit 的 sensor_height 必须跟着变；
+      C（抽稀网格碰撞）：**已查清**：spawn 正常但传感器一条数据都没有 —— 根因是 ODE 的
+         ray-vs-trimesh 是 O(#三角面) 的，30000 条射线 × 3000 面 = 9×10⁷ 次/帧 @10 Hz
+         ⇒ gzserver 在"打一帧射线"里出不来（传感器回调永不返回），不是插件没挂上。
+    倾斜感知链（**全部只对本槽位生效**，默认模型逐字节不变）：
+      · linefit：`sensor_height` = 雷达离地（0.2595 + raise）、`gravity_aligned_frame` = base_link
+        （雷达斜 30° ⇒ 传感器系的 z 不再是"高度"）—— 见 `config/segmentation_sim_robot11.yaml`
+      · pointcloud_to_laserscan：`target_frame` = base_link（高度带改在重力对齐系里量）
+        —— 见 `config/laserscan_params_robot11.yaml`
+      · LIO 外参：**不改**。IMU 与雷达同壳、只差 0.05 m 平移（`extrinsic_T=[0,0,0.05]`,
+        `extrinsic_R=I` 逐字节沿用），IMU 姿态里的 30° 由 LIO 自己估出来，
+        `odom→base_link` 由 small_point_lio 用 `base_link→livox_frame` 的 TF 精确换算。
   ── ⚠️ 上游的 <collision> 全被替换掉了（这是本槽位最关键的一处偏离） ────────
     上游 12 个 link 的 collision **全部是 mesh**，其中 `body` = 2,078,226 面。
@@ -42,9 +66,21 @@
   <xacro:arg name="xyz" default="0 0 0"/>
   <xacro:arg name="rpy" default="0 0 0"/>
-  <!-- 【我们加的】雷达 30° 安装的旋转；默认 = SolidWorks CSV 的 roll 形式。
+  <!-- 【我们加的】雷达 30° 安装的旋转；默认 = SolidWorks CSV 的 roll 形式
+       （用户 2026-10-07 **按实物确认：是绕 roll**；pitch 只作对照开关）。
        pitch 形式 = "0 -0.523598775598293 0"。两者对 360° 雷达几何等价（差一个绕 z 的旋转）。 -->
   <xacro:arg name="livox_tilt_rpy" default="-0.523598775598293 0 0"/>
-  <!-- ==================== link body ==================== -->
-  <link name="body">
+  <!-- 【我们加的｜B 方案，默认 0 = 与上游逐字相同】把雷达（连同 IMU）整体抬高的米数。
+       用途：实测"不做碰撞开口、直接把雷达抬到顶板上方"这条仿真适配路（docs/robot_models.md §11）。
+       ⚠️ 抬高会改变雷达离地高度 ⇒ linefit 的 sensor_height 必须同步 = 0.2595 + livox_raise_m
+       （launch 里由 robot:=robot11 分支**算出来**注入，不是手抄）。默认 0 ⇒ 一切不变。 -->
+  <xacro:arg name="livox_raise_m" default="0"/>
+  <!-- xacro 的表达式里**不能直接写 arg 名**（实测报 name 'livox_raise_m' is not defined）
+       ⇒ 按标准写法先绑成 property 再进表达式。 -->
+  <xacro:property name="livox_raise_m_p" value="$(arg livox_raise_m)"/>
+  <!-- 【我们加的｜改名】上游根 link `body` → `base_link`（原因见文件头第 3 条）：
+       本栈契约帧名是 base_link；不改名的实测后果 = TF 断树、LIO 发不出 /odom、
+       p2l 丢光整条点云。上游 SolidWorks CSV 里这个 link 本来就叫 base_link。 -->
+  <!-- ==================== link base_link ==================== -->
+  <link name="base_link">
     <!-- 【上游原样】inertial -->
     <inertial>
@@ -60,21 +96,315 @@
     </visual>
     <!-- 【我们加的｜替换】上游这里是 mesh collision；按 Phase 1 实测换掉（原因见文件头） -->
-    <!-- body：4 个 box = DP 最优 z 分段包络（覆盖率 1.000 / 总体积 0.065121 m³，网格凸包 0.0595 m³）
-         生成：robot11_make_collision_assets.py，清单：robot11_description/inventory/collision_assets.json -->
-    <collision>
-      <origin xyz="0 0 -0.005444" rpy="0 0 0"/>
-      <geometry><box size="0.6 0.6 0.085"/></geometry>
-    </collision>
-    <collision>
-      <origin xyz="0 0 0.072056" rpy="0 0 0"/>
-      <geometry><box size="0.553269 0.549539 0.07"/></geometry>
-    </collision>
-    <collision>
-      <origin xyz="0 -0.00634 0.124556" rpy="0 0 0"/>
-      <geometry><box size="0.532413 0.334483 0.035"/></geometry>
-    </collision>
-    <collision>
-      <origin xyz="0 -0.014821 0.177528" rpy="0 0 0"/>
-      <geometry><box size="0.285 0.346467 0.070944"/></geometry>
+    <!-- base_link：**A 方案 = DP box 减去"雷达视锥"**（76 个 box，Phase 3 采用）
+         为什么：雷达原点 z=0.157 落在第 4 个 DP box **内部**（box 顶 0.213）⇒ 实心包络
+           把凹槽填实 ⇒ 每条射线先打到盒内壁（Phase 2 实测 75.5% 的点 r<0.12 m、
+           `/segmentation/ground` 529 点/帧、LIO 无 `/odom`）。挖掉视锥后离线实测：
+           自击<0.12 m = 0%、看见地面 = 25.2%（30000 条与 Gazebo 同源的射线）。
+         生成：robot11_livox_fov.py —emit-carved；清单：inventory/livox_fov_boxes.json
+         参数：锥半角 100.22°、半径 0.50 m、内清空 0.05 m、体素 [0.015, 0.015, 0.01535] m、倾角轴 roll
+         ⚠️ 这是**仿真侧适配**（偏离上游 CAD 的碰撞几何），逐条登记在 docs/robot_models.md §11 -->
+    <collision>
+      <origin xyz="0.000000 0.000000 -0.040269" rpy="0 0 0"/>
+      <geometry><box size="0.600000 0.600000 0.015350"/></geometry>
+    </collision>
+    <collision>
+      <origin xyz="0.000000 -0.007500 -0.024920" rpy="0 0 0"/>
+      <geometry><box size="0.600000 0.585000 0.015350"/></geometry>
+    </collision>
+    <collision>
+      <origin xyz="0.000000 -0.015000 -0.009570" rpy="0 0 0"/>
+      <geometry><box size="0.600000 0.570000 0.015350"/></geometry>
+    </collision>
+    <collision>
+      <origin xyz="0.000000 -0.030000 0.005780" rpy="0 0 0"/>
+      <geometry><box size="0.600000 0.540000 0.015350"/></geometry>
+    </collision>
+    <collision>
+      <origin xyz="0.000000 -0.037500 0.021129" rpy="0 0 0"/>
+      <geometry><box size="0.600000 0.525000 0.015350"/></geometry>
+    </collision>
+    <collision>
+      <origin xyz="0.000000 -0.052500 0.036479" rpy="0 0 0"/>
+      <geometry><box size="0.600000 0.495000 0.015350"/></geometry>
+    </collision>
+    <collision>
+      <origin xyz="0.000000 -0.037500 0.051829" rpy="0 0 0"/>
+      <geometry><box size="0.540000 0.465000 0.015350"/></geometry>
+    </collision>
+    <collision>
+      <origin xyz="0.000000 -0.052500 0.067178" rpy="0 0 0"/>
+      <geometry><box size="0.540000 0.435000 0.015350"/></geometry>
+    </collision>
+    <collision>
+      <origin xyz="0.000000 -0.067500 0.082528" rpy="0 0 0"/>
+      <geometry><box size="0.540000 0.405000 0.015350"/></geometry>
+    </collision>
+    <collision>
+      <origin xyz="0.000000 -0.075000 0.097878" rpy="0 0 0"/>
+      <geometry><box size="0.540000 0.390000 0.015350"/></geometry>
+    </collision>
+    <collision>
+      <origin xyz="0.000000 -0.045000 0.113227" rpy="0 0 0"/>
+      <geometry><box size="0.540000 0.270000 0.015350"/></geometry>
+    </collision>
+    <collision>
+      <origin xyz="0.000000 -0.060000 0.128577" rpy="0 0 0"/>
+      <geometry><box size="0.540000 0.240000 0.015350"/></geometry>
+    </collision>
+    <collision>
+      <origin xyz="0.000000 -0.060000 0.143927" rpy="0 0 0"/>
+      <geometry><box size="0.300000 0.270000 0.015350"/></geometry>
+    </collision>
+    <collision>
+      <origin xyz="0.000000 -0.075000 0.159276" rpy="0 0 0"/>
+      <geometry><box size="0.300000 0.240000 0.015350"/></geometry>
+    </collision>
+    <collision>
+      <origin xyz="0.000000 -0.090000 0.174626" rpy="0 0 0"/>
+      <geometry><box size="0.300000 0.210000 0.015350"/></geometry>
+    </collision>
+    <collision>
+      <origin xyz="0.000000 -0.112500 0.189976" rpy="0 0 0"/>
+      <geometry><box size="0.300000 0.165000 0.015350"/></geometry>
+    </collision>
+    <collision>
+      <origin xyz="0.000000 -0.127500 0.205325" rpy="0 0 0"/>
+      <geometry><box size="0.300000 0.135000 0.015350"/></geometry>
+    </collision>
+    <collision>
+      <origin xyz="0.000000 0.247500 0.005780" rpy="0 0 0"/>
+      <geometry><box size="0.570000 0.015000 0.015350"/></geometry>
+    </collision>
+    <collision>
+      <origin xyz="0.000000 0.202500 0.036479" rpy="0 0 0"/>
+      <geometry><box size="0.570000 0.015000 0.015350"/></geometry>
+    </collision>
+    <collision>
+      <origin xyz="0.007500 0.292500 -0.024920" rpy="0 0 0"/>
+      <geometry><box size="0.555000 0.015000 0.015350"/></geometry>
+    </collision>
+    <collision>
+      <origin xyz="0.007500 0.232500 0.021129" rpy="0 0 0"/>
+      <geometry><box size="0.525000 0.015000 0.015350"/></geometry>
+    </collision>
+    <collision>
+      <origin xyz="0.000000 0.277500 -0.009570" rpy="0 0 0"/>
+      <geometry><box size="0.510000 0.015000 0.015350"/></geometry>
+    </collision>
+    <collision>
+      <origin xyz="0.000000 0.142500 0.082528" rpy="0 0 0"/>
+      <geometry><box size="0.510000 0.015000 0.015350"/></geometry>
+    </collision>
+    <collision>
+      <origin xyz="0.000000 0.217500 0.036479" rpy="0 0 0"/>
+      <geometry><box size="0.480000 0.015000 0.015350"/></geometry>
+    </collision>
+    <collision>
+      <origin xyz="0.000000 0.172500 0.067178" rpy="0 0 0"/>
+      <geometry><box size="0.480000 0.015000 0.015350"/></geometry>
+    </collision>
+    <collision>
+      <origin xyz="0.000000 0.097500 0.113227" rpy="0 0 0"/>
+      <geometry><box size="0.480000 0.015000 0.015350"/></geometry>
+    </collision>
+    <collision>
+      <origin xyz="0.000000 0.067500 0.128577" rpy="0 0 0"/>
+      <geometry><box size="0.480000 0.015000 0.015350"/></geometry>
+    </collision>
+    <collision>
+      <origin xyz="0.000000 0.262500 0.005780" rpy="0 0 0"/>
+      <geometry><box size="0.450000 0.015000 0.015350"/></geometry>
+    </collision>
+    <collision>
+      <origin xyz="0.000000 0.127500 0.097878" rpy="0 0 0"/>
+      <geometry><box size="0.450000 0.015000 0.015350"/></geometry>
+    </collision>
+    <collision>
+      <origin xyz="0.000000 0.247500 0.021129" rpy="0 0 0"/>
+      <geometry><box size="0.420000 0.015000 0.015350"/></geometry>
+    </collision>
+    <collision>
+      <origin xyz="0.000000 0.202500 0.051829" rpy="0 0 0"/>
+      <geometry><box size="0.420000 0.015000 0.015350"/></geometry>
+    </collision>
+    <collision>
+      <origin xyz="0.000000 0.157500 0.082528" rpy="0 0 0"/>
+      <geometry><box size="0.420000 0.015000 0.015350"/></geometry>
+    </collision>
+    <collision>
+      <origin xyz="0.000000 0.082500 0.128577" rpy="0 0 0"/>
+      <geometry><box size="0.420000 0.015000 0.015350"/></geometry>
+    </collision>
+    <collision>
+      <origin xyz="0.000000 0.292500 -0.009570" rpy="0 0 0"/>
+      <geometry><box size="0.360000 0.015000 0.015350"/></geometry>
+    </collision>
+    <collision>
+      <origin xyz="0.000000 0.232500 0.036479" rpy="0 0 0"/>
+      <geometry><box size="0.360000 0.015000 0.015350"/></geometry>
+    </collision>
+    <collision>
+      <origin xyz="0.000000 0.187500 0.067178" rpy="0 0 0"/>
+      <geometry><box size="0.360000 0.015000 0.015350"/></geometry>
+    </collision>
+    <collision>
+      <origin xyz="0.000000 0.142500 0.097878" rpy="0 0 0"/>
+      <geometry><box size="0.360000 0.015000 0.015350"/></geometry>
+    </collision>
+    <collision>
+      <origin xyz="0.000000 0.172500 0.082528" rpy="0 0 0"/>
+      <geometry><box size="0.330000 0.015000 0.015350"/></geometry>
+    </collision>
+    <collision>
+      <origin xyz="0.000000 0.277500 0.005780" rpy="0 0 0"/>
+      <geometry><box size="0.300000 0.015000 0.015350"/></geometry>
+    </collision>
+    <collision>
+      <origin xyz="0.000000 0.217500 0.051829" rpy="0 0 0"/>
+      <geometry><box size="0.300000 0.015000 0.015350"/></geometry>
+    </collision>
+    <collision>
+      <origin xyz="0.007500 -0.022500 0.189976" rpy="0 0 0"/>
+      <geometry><box size="0.285000 0.015000 0.015350"/></geometry>
+    </collision>
+    <collision>
+      <origin xyz="0.000000 0.262500 0.021129" rpy="0 0 0"/>
+      <geometry><box size="0.270000 0.015000 0.015350"/></geometry>
+    </collision>
+    <collision>
+      <origin xyz="0.000000 0.202500 0.067178" rpy="0 0 0"/>
+      <geometry><box size="0.270000 0.015000 0.015350"/></geometry>
+    </collision>
+    <collision>
+      <origin xyz="0.000000 0.157500 0.097878" rpy="0 0 0"/>
+      <geometry><box size="0.270000 0.015000 0.015350"/></geometry>
+    </collision>
+    <collision>
+      <origin xyz="0.000000 0.082500 0.143927" rpy="0 0 0"/>
+      <geometry><box size="0.270000 0.015000 0.015350"/></geometry>
+    </collision>
+    <collision>
+      <origin xyz="0.000000 0.052500 0.159276" rpy="0 0 0"/>
+      <geometry><box size="0.240000 0.015000 0.015350"/></geometry>
+    </collision>
+    <collision>
+      <origin xyz="0.000000 0.022500 0.174626" rpy="0 0 0"/>
+      <geometry><box size="0.240000 0.015000 0.015350"/></geometry>
+    </collision>
+    <collision>
+      <origin xyz="0.000000 -0.052500 0.205325" rpy="0 0 0"/>
+      <geometry><box size="0.240000 0.015000 0.015350"/></geometry>
+    </collision>
+    <collision>
+      <origin xyz="0.000000 0.247500 0.036479" rpy="0 0 0"/>
+      <geometry><box size="0.210000 0.015000 0.015350"/></geometry>
+    </collision>
+    <collision>
+      <origin xyz="0.000000 0.187500 0.082528" rpy="0 0 0"/>
+      <geometry><box size="0.210000 0.015000 0.015350"/></geometry>
+    </collision>
+    <collision>
+      <origin xyz="-0.105000 0.112500 0.113227" rpy="0 0 0"/>
+      <geometry><box size="0.180000 0.015000 0.015350"/></geometry>
+    </collision>
+    <collision>
+      <origin xyz="0.105000 0.112500 0.113227" rpy="0 0 0"/>
+      <geometry><box size="0.180000 0.015000 0.015350"/></geometry>
+    </collision>
+    <collision>
+      <origin xyz="0.000000 0.067500 0.159276" rpy="0 0 0"/>
+      <geometry><box size="0.180000 0.015000 0.015350"/></geometry>
+    </collision>
+    <collision>
+      <origin xyz="0.000000 -0.007500 0.189976" rpy="0 0 0"/>
+      <geometry><box size="0.180000 0.015000 0.015350"/></geometry>
+    </collision>
+    <collision>
+      <origin xyz="0.000000 0.232500 0.051829" rpy="0 0 0"/>
+      <geometry><box size="0.150000 0.015000 0.015350"/></geometry>
+    </collision>
+    <collision>
+      <origin xyz="0.000000 0.172500 0.097878" rpy="0 0 0"/>
+      <geometry><box size="0.150000 0.015000 0.015350"/></geometry>
+    </collision>
+    <collision>
+      <origin xyz="0.000000 0.037500 0.174626" rpy="0 0 0"/>
+      <geometry><box size="0.150000 0.015000 0.015350"/></geometry>
+    </collision>
+    <collision>
+      <origin xyz="-0.097500 0.097500 0.128577" rpy="0 0 0"/>
+      <geometry><box size="0.135000 0.015000 0.015350"/></geometry>
+    </collision>
+    <collision>
+      <origin xyz="0.097500 0.097500 0.128577" rpy="0 0 0"/>
+      <geometry><box size="0.135000 0.015000 0.015350"/></geometry>
+    </collision>
+    <collision>
+      <origin xyz="-0.090000 0.127500 0.113227" rpy="0 0 0"/>
+      <geometry><box size="0.120000 0.015000 0.015350"/></geometry>
+    </collision>
+    <collision>
+      <origin xyz="0.000000 0.157500 0.113227" rpy="0 0 0"/>
+      <geometry><box size="0.120000 0.015000 0.015350"/></geometry>
+    </collision>
+    <collision>
+      <origin xyz="0.090000 0.127500 0.113227" rpy="0 0 0"/>
+      <geometry><box size="0.120000 0.015000 0.015350"/></geometry>
+    </collision>
+    <collision>
+      <origin xyz="0.000000 0.217500 0.067178" rpy="0 0 0"/>
+      <geometry><box size="0.090000 0.015000 0.015350"/></geometry>
+    </collision>
+    <collision>
+      <origin xyz="-0.060000 0.142500 0.113227" rpy="0 0 0"/>
+      <geometry><box size="0.090000 0.015000 0.015350"/></geometry>
+    </collision>
+    <collision>
+      <origin xyz="0.060000 0.142500 0.113227" rpy="0 0 0"/>
+      <geometry><box size="0.090000 0.015000 0.015350"/></geometry>
+    </collision>
+    <collision>
+      <origin xyz="-0.075000 0.112500 0.128577" rpy="0 0 0"/>
+      <geometry><box size="0.090000 0.015000 0.015350"/></geometry>
+    </collision>
+    <collision>
+      <origin xyz="0.075000 0.112500 0.128577" rpy="0 0 0"/>
+      <geometry><box size="0.090000 0.015000 0.015350"/></geometry>
+    </collision>
+    <collision>
+      <origin xyz="0.000000 -0.037500 0.205325" rpy="0 0 0"/>
+      <geometry><box size="0.090000 0.015000 0.015350"/></geometry>
+    </collision>
+    <collision>
+      <origin xyz="0.000000 0.292500 0.005780" rpy="0 0 0"/>
+      <geometry><box size="0.060000 0.015000 0.015350"/></geometry>
+    </collision>
+    <collision>
+      <origin xyz="-0.060000 0.097500 0.143927" rpy="0 0 0"/>
+      <geometry><box size="0.060000 0.015000 0.015350"/></geometry>
+    </collision>
+    <collision>
+      <origin xyz="0.060000 0.097500 0.143927" rpy="0 0 0"/>
+      <geometry><box size="0.060000 0.015000 0.015350"/></geometry>
+    </collision>
+    <collision>
+      <origin xyz="0.000000 0.007500 0.189976" rpy="0 0 0"/>
+      <geometry><box size="0.060000 0.015000 0.015350"/></geometry>
+    </collision>
+    <collision>
+      <origin xyz="-0.060000 0.127500 0.128577" rpy="0 0 0"/>
+      <geometry><box size="0.030000 0.015000 0.015350"/></geometry>
+    </collision>
+    <collision>
+      <origin xyz="0.060000 0.127500 0.128577" rpy="0 0 0"/>
+      <geometry><box size="0.030000 0.015000 0.015350"/></geometry>
+    </collision>
+    <collision>
+      <origin xyz="-0.030000 0.082500 0.159276" rpy="0 0 0"/>
+      <geometry><box size="0.030000 0.015000 0.015350"/></geometry>
+    </collision>
+    <collision>
+      <origin xyz="0.030000 0.082500 0.159276" rpy="0 0 0"/>
+      <geometry><box size="0.030000 0.015000 0.015350"/></geometry>
     </collision>
   </link>
@@ -262,8 +592,34 @@
     </visual>
     <!-- 【我们加的｜替换】上游这里是 mesh collision；按 Phase 1 实测换掉（原因见文件头） -->
-    <!-- l10：**解析 box**（= 源 mesh l10.STL 的包围盒；理由见下） -->
+    <!-- l10：**细碰撞盒 7 个**（Phase 3 换掉单包围盒；离雷达最近面 0.1246 m，单包围盒时 0.0993 m）
+         生成：robot11_livox_fov.py —emit-turret-boxes；清单：inventory/turret_boxes.json
+         方法：voxel + binary_closing(3x3x3) + binary_fill_holes + 贪心 box 分解；体素 15 mm（上游 mesh 不水密 ⇒ 只能"实心近似"） -->
     <collision>
       <origin xyz="-0.063500 0.019350 0.002895" rpy="0 0 0"/>
-      <geometry><box size="0.147000 0.137900 0.070566"/></geometry>
+      <geometry><box size="0.125600 0.118320 0.016113"/></geometry>
+    </collision>
+    <collision>
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