Commit message: fix(bringup): robot11 —— 更正骗人的横幅、补运行期接线证据、视觉档位开关（默认抽稀）、GUI 代价实测工具
缺陷 ③（用户 2026-10-07）：launch 横幅写「⚠️ linefit 参数**没有**跟着切（sensor_height 仍是
0.226、gravity_aligned_frame 仍是 ""）」，而 Phase 3 其实**已经**用 _RobotSlotFile.slot_map 切到
segmentation_sim_robot11.yaml 了 ⇒ 横幅在骗人，用户照它排查就查错方向。
根因：横幅写的是**意图**，不是**生效值**。

· 新增 _YamlKeysReadout / _SelfMaskReadout 两个 Substitution：横幅在**运行时**把真正递给节点的
  那份 YAML 读出来、把键值打进日志 ⇒ 横幅与「节点实际读到的文件」不可能再分叉。
  运行期证据（同一次跑）：横幅打印
    sensor_height=0.2595, gravity_aligned_frame="", input_topic=/livox/lidar/pointcloud,
    ground_output_topic=segmentation/ground  ← .../config/segmentation_sim_robot11.yaml
    self_mask_enable=true, 近场死区 r<=0.2416 m（z>=-0.2295）, 113 个 collision AABB ← ...
  节点侧：ros2 param get /ground_segmentation sensor_height → Double value is: 0.2595；
    gravity_aligned_frame → 空串；self_mask_enable → True；self_mask_boxes → 678 个数（113 盒）。
· 横幅里「lio_tf_adapter 杆臂 = T_imu←base_link（含 30° 旋转补偿）」在本配置下是**误导**：
  lio:=small_point_lio 时该节点**按设计不启动**（单 odom→base_link 发布者契约；
  实测 ros2 param get /lio_tf_adapter xyz → Node not found），杆臂由 LIO 自己用
  lookupTransform(lidar_frame,"base_link") 做相似变换；而 Phase 3 已把 body_to_livox 的 rpy 改成 0
  ⇒ 运行期 TF base_link→livox_frame 是**纯平移** [0.001,0.131,0.157]、RPY 0（tf2_echo 实测）
  ⇒ 旋转补偿在本槽位**不需要**。横幅已改成说明这一点。

缺陷 ①（同一跑的 gzclient exit -9 / rviz2 黑屏）：视觉一直是上游原始 STL（12 个 mesh 合计
2,821,320 面 / 141.07 MB，其中 base_link.STL 一项 99 MiB / 2,078,226 面）。实测 rviz2 峰值 RSS
随视觉档位在 **243 MiB ↔ 1,381 MiB** 之间（+1.14 GB）。

· xacro 新增 `visual_decimated`（默认 false = 上游原始 STL，与 Phase 1~3 逐字节相同）：
  只换 `<visual>` 的 mesh 文件名，`<collision>`/`<sensor>`/`<plugin>`/inertial 一个字节不动。
· launch 新增 `robot11_visual:=decimated|full`（**默认 decimated**），只对 robot:=robot11 生效；
  decimated 复用 Phase 1 已入库的抽稀件 meshes/generated/*_collision.stl（9,700 面 / 0.486 MB，
  bbox 与原件差 ≤3 mm、单位/原点不变）。
  ⚠️ 已知重叠：Phase 5（另一路）正在做**更好的**视觉 LOD（meshes/decimated/ + 量化验收 +
  generator 重算本 xacro）。本 commit 的 `visual_decimated` 布尔 arg 已被对方的
  check_robot11_visual_slot.py 列为兼容别名（优先级：显式传的赢；都不传 ⇒ decimated）。

GUI 代价实测（新增 tools/scripts/regress/robot11_gui_bench.sh；Xvfb 3200x1200 + llvmpipe 软件 GL，
窗口从 gzclient/rviz2 都起来开始计 50 s，RSS 每 1 s 采样）：
  | 指标 | full | decimated |
  | gzclient 峰值 RSS | 474 MiB | 474 MiB |
  | gzserver 峰值 RSS | 3202 MiB（无头对照 3112 MiB） | 3202 MiB |
  | rviz2 峰值 RSS | 1381 MiB | 243 MiB |
  | 存活 | gzclient/rviz2 都活满，无死亡行 | 同 |
  | rviz2 窗口内非黑像素/颜色数 | 0.5768 / 1023 | 0.5768 / 1438 |
  ⚠️ 软件 GL ⇒ 渲染吞吐不可测（不代表真 GPU）；本轮**没有复现**用户的 gzclient SIGKILL。
  ⚠️ gzclient 的 RSS 不随视觉档位变 ⇒ 真正被降下来的是 rviz2。

工具：run_robot_model_probe.sh 增加 self_mask_* 回读、TF 安装几何回读、SLOPE_PROBE_ARGS 挂钩，
以及**端口先探测再占用**（残留 gzserver 占着 11350+hash%500 时新 gzserver 会直接 exit 255，
实测踩到两次；显式给 GAZEBO_MASTER_URI 时完全听调用方的）。

File: src/rm_nav_bringup/urdf/sentry_robot_robot11_sim.xacro (robot description, xacro)
@@ -78,4 +78,21 @@
        ⇒ 按标准写法先绑成 property 再进表达式。 -->
   <xacro:property name="livox_raise_m_p" value="$(arg livox_raise_m)"/>
+  <!-- 【我们加的｜Phase 4，默认 false = 与 Phase 1~3 逐字节相同】视觉 mesh 用哪一档。
+       true  = 复用 Phase 1 已经生成并入库的**抽稀件** `meshes/generated/<link>_collision.stl`
+               （VTK quadric decimation：base_link 2,078,226 → 3,000 面、l11 176,459 → 1,200 面；
+                bbox 与原件差 ≤3 mm，单位/原点不变 ⇒ 米制与几何位置都不改）。
+       false = 上游原始 STL（`meshes/<link>.STL`，base_link 那份 99 MiB / 207.8 万面）。
+       为什么需要：用户 2026-10-07 带 GUI 跑 robot:=robot11 时 **gzclient 被 SIGKILL（exit -9）**、
+       rviz2 黑屏 —— 就是这一档的渲染/内存代价（docs/robot_models.md §12 有实测对照）。
+       ⚠️ 只换 `<visual>`：`<collision>`（76 box + 云台细盒 + cylinder）一个字节都不动
+       ⇒ 物理/感知/契约完全不变；`robot:=robot11` 之外的模型根本不引用这两个 property。 -->
+  <xacro:arg name="visual_decimated" default="false"/>
+  <xacro:property name="visual_decimated_p" value="$(arg visual_decimated)"/>
+  <!-- ⚠️ xacro 会把 `"true"` 这个 arg **转成 Python 的 bool True**（实测：`${vd_p}` 打印 True），
+       所以这里必须 `str(...).lower()` 归一化，不能直接和字符串 'true' 比。 -->
+  <xacro:property name="visual_dir"
+      value="${'generated' if str(visual_decimated_p).lower() in ('true', '1') else 'meshes'}"/>
+  <xacro:property name="visual_ext"
+      value="${'_collision.stl' if str(visual_decimated_p).lower() in ('true', '1') else '.STL'}"/>
   <!-- 【我们加的｜改名】上游根 link `body` → `base_link`（原因见文件头第 3 条）：
        本栈契约帧名是 base_link；不改名的实测后果 = TF 断树、LIO 发不出 /odom、
@@ -92,5 +109,5 @@
     <visual>
       <origin xyz="0 0 0" rpy="0 0 0"/>
-      <geometry><mesh filename="package://robot11/meshes/base_link.STL"/></geometry>
+      <geometry><mesh filename="package://robot11/${visual_dir}/base_link${visual_ext}"/></geometry>
       <material name=""><color rgba="0.792156862745098 0.819607843137255 0.933333333333333 1"/></material>
     </visual>
@@ -420,5 +437,5 @@
     <visual>
       <origin xyz="0 0 0" rpy="0 0 0"/>
-      <geometry><mesh filename="package://robot11/meshes/l2.STL"/></geometry>
+      <geometry><mesh filename="package://robot11/${visual_dir}/l2${visual_ext}"/></geometry>
       <material name=""><color rgba="0.792156862745098 0.819607843137255 0.933333333333333 1"/></material>
     </visual>
@@ -441,5 +458,5 @@
     <visual>
       <origin xyz="0 0 0" rpy="0 0 0"/>
-      <geometry><mesh filename="package://robot11/meshes/l6.STL"/></geometry>
+      <geometry><mesh filename="package://robot11/${visual_dir}/l6${visual_ext}"/></geometry>
       <material name=""><color rgba="0.792156862745098 0.819607843137255 0.933333333333333 1"/></material>
     </visual>
@@ -462,5 +479,5 @@
     <visual>
       <origin xyz="0 0 0" rpy="0 0 0"/>
-      <geometry><mesh filename="package://robot11/meshes/l3.STL"/></geometry>
+      <geometry><mesh filename="package://robot11/${visual_dir}/l3${visual_ext}"/></geometry>
       <material name=""><color rgba="0.792156862745098 0.819607843137255 0.933333333333333 1"/></material>
     </visual>
@@ -483,5 +500,5 @@
     <visual>
       <origin xyz="0 0 0" rpy="0 0 0"/>
-      <geometry><mesh filename="package://robot11/meshes/l7.STL"/></geometry>
+      <geometry><mesh filename="package://robot11/${visual_dir}/l7${visual_ext}"/></geometry>
       <material name=""><color rgba="0.792156862745098 0.819607843137255 0.933333333333333 1"/></material>
     </visual>
@@ -504,5 +521,5 @@
     <visual>
       <origin xyz="0 0 0" rpy="0 0 0"/>
-      <geometry><mesh filename="package://robot11/meshes/l4.STL"/></geometry>
+      <geometry><mesh filename="package://robot11/${visual_dir}/l4${visual_ext}"/></geometry>
       <material name=""><color rgba="0.792156862745098 0.819607843137255 0.933333333333333 1"/></material>
     </visual>
@@ -525,5 +542,5 @@
     <visual>
       <origin xyz="0 0 0" rpy="0 0 0"/>
-      <geometry><mesh filename="package://robot11/meshes/l8.STL"/></geometry>
+      <geometry><mesh filename="package://robot11/${visual_dir}/l8${visual_ext}"/></geometry>
       <material name=""><color rgba="0.792156862745098 0.819607843137255 0.933333333333333 1"/></material>
     </visual>
@@ -546,5 +563,5 @@
     <visual>
       <origin xyz="0 0 0" rpy="0 0 0"/>
-      <geometry><mesh filename="package://robot11/meshes/l5.STL"/></geometry>
+      <geometry><mesh filename="package://robot11/${visual_dir}/l5${visual_ext}"/></geometry>
       <material name=""><color rgba="0.792156862745098 0.819607843137255 0.933333333333333 1"/></material>
     </visual>
@@ -567,5 +584,5 @@
     <visual>
       <origin xyz="0 0 0" rpy="0 0 0"/>
-      <geometry><mesh filename="package://robot11/meshes/l9.STL"/></geometry>
+      <geometry><mesh filename="package://robot11/${visual_dir}/l9${visual_ext}"/></geometry>
       <material name=""><color rgba="0.792156862745098 0.819607843137255 0.933333333333333 1"/></material>
     </visual>
@@ -588,5 +605,5 @@
     <visual>
       <origin xyz="0 0 0" rpy="0 0 0"/>
-      <geometry><mesh filename="package://robot11/meshes/l10.STL"/></geometry>
+      <geometry><mesh filename="package://robot11/${visual_dir}/l10${visual_ext}"/></geometry>
       <material name=""><color rgba="0.792156862745098 0.819607843137255 0.933333333333333 1"/></material>
     </visual>
@@ -635,5 +652,5 @@
     <visual>
       <origin xyz="0 0 0" rpy="0 0 0"/>
-      <geometry><mesh filename="package://robot11/meshes/l11.STL"/></geometry>
+      <geometry><mesh filename="package://robot11/${visual_dir}/l11${visual_ext}"/></geometry>
       <material name=""><color rgba="0.792156862745098 0.819607843137255 0.933333333333333 1"/></material>
     </visual>
@@ -742,5 +759,5 @@
     <visual>
       <origin xyz="0 0 0" rpy="0 0 0"/>
-      <geometry><mesh filename="package://robot11/meshes/l12.STL"/></geometry>
+      <geometry><mesh filename="package://robot11/${visual_dir}/l12${visual_ext}"/></geometry>
       <material name=""><color rgba="0.792156862745098 0.819607843137255 0.933333333333333 1"/></material>
     </visual>

Commit message: feat(robot11): `decimated` 档改指**专用视觉 LOD** + 开关契约检查工具 + 三处不再骗人的横幅（Phase 5）
接上一个提交：抽稀件与清单入库后，把 `robot11_visual:=decimated`（默认）真正指过去。

· `tools/scripts/regress/robot11_make_sim_xacro.py`（**生成器接管**）：
  - `sentry_robot_robot11_sim.xacro` 的正确改法是改生成器再重跑，不是手改生成物
    （文件头自己写着"本文件是生成的，不要手改"）。Phase 4 手改进生成物的那段 arg/property
    按同一语义搬进生成器：`robot11_visual`（decimated|full，默认 decimated）为主开关，
    `visual_decimated`（Phase 4 的布尔别名）保留为兼容别名，**非空时它赢**（命令行优先于默认值）；
  - 档位解析：`visual_dir` = `meshes/decimated` | `meshes`，`visual_ext` = `.stl` | `.STL`；
    每个 link 的 `<visual><geometry><mesh filename>` 由这两个 property 拼出来；
  - **前置校验**：视觉清单缺失或 `all_ok=false` ⇒ 生成器**直接报错**（不生成"看起来对但没人验证过"的模型）；
    清单里的三角形数/字节数/几个大头会被写进生成物的文件头（provenance 是构造性的）。
· `urdf/sentry_robot_robot11_sim.xacro`：重跑生成器得到（除 `<visual>` 的 mesh 文件名外
  与上一版**逐元素相同** —— 由下面的检查工具 A1/G5 断言）。
· `tools/scripts/regress/check_robot11_visual_slot.py`（新增，21 项断言，真的跑 `xacro` 渲染两档）：
  A1「两档 URDF 除 visual mesh 文件名外**逐字节相同**」、B1 `<visual><origin>` 逐字相同、
  C1 引用文件都存在、D1 没有 `<mesh scale=...>`、E1~E3 三角形预算、F1 清单↔磁盘 sha256 一致、
  F2~F5 全部容差、**G1 质量合计 9.5521 kg / G2 `body_to_livox` xyz 逐字不变 / G3 四个转向关节
  ±0.1821345596729 / G4 轮 collision 仍是 cylinder r=0.058 / G5 collision 元素个数相同**、
  H1~H4 默认值与两个 arg 的优先级。当前**全绿**。
· `launch/bringup_sim.launch.py`：只改**文案**（三处），不带行为变化 ——
  `robot11_visual` 的 description、xacro 命令处的注释、robot11 模型横幅里"decimated = 复用
  Phase 1 的抽稀件 generated/*_collision.stl（少 3 个数量级）"这句**已经过期**的话
  （现在指向 `meshes/decimated/`，且 Phase 4 的 GUI 内存结论在本轮没有被复现，见 §13.4.3）。
  `--show-args` 已实测仍正常（rc=0，新文案在里面）。

`<collision>` / `<inertial>` / `<sensor>` / `<plugin>` 一个字节没动 ⇒ 物理、感知、契约不变；
`robot:=robot11` 之外的模型不引用这两个 property ⇒ 默认模型逐字节不变。

File: src/rm_nav_bringup/urdf/sentry_robot_robot11_sim.xacro (robot description, xacro)
@@ -58,5 +58,14 @@
       · 峰值内存恒 **759 MB vs 基线 172 MB**
     ⇒ 替换为：`body` = 4 个 box（DP 最优分段包络，覆盖率 1.000、总体积只比凸包胖 9.4%）；
-      轮 = cylinder；其余 = 抽稀件。**`<visual>` 仍然是原始 mesh，视觉零损失。**
+      轮 = cylinder；其余 = 抽稀件。
+  ── Phase 5（2026-10-07）：把 `<visual>` 也换档（**这才是"带 GUI 放得进仿真"的那一步**）──
+    Phase 1~3 只改了**碰撞**侧，**视觉**侧一直是上游原始 STL：整车 2,870,498 面，其中
+    `base_link.STL` 一项 2,078,226 面 / 99 MiB。用户 2026-10-07 带 GUI 跑 ⇒ **gzclient 被内核
+    SIGKILL（exit -9）**、rviz2 黑屏 —— 因为 gzclient 会把每个 `<visual>` 网格整份渲进 OGRE。
+    Phase 5 按公开的标准管线（视觉/碰撞分离 + QEM 抽稀 + 量化验证，引用见 docs/robot_models.md
+    §13.2）生成**视觉 LOD**：每 link ≤ 50k 面、整车 ≤ 200k 面，逐 mesh 量化"包围盒差 /
+    单向表面误差 p99,max / 三视剪影 IoU / 边界边数"，全部落在
+    `robot11_description/inventory/visual_decimation.json`。
+    开关：`robot11_visual:=decimated`（**默认**）| `full`；`<collision>` 与 `<inertial>` 不动。
 -->
 <robot name="sentry" xmlns:xacro="http://ros.org/wiki/xacro">
@@ -78,21 +87,36 @@
        ⇒ 按标准写法先绑成 property 再进表达式。 -->
   <xacro:property name="livox_raise_m_p" value="$(arg livox_raise_m)"/>
-  <!-- 【我们加的｜Phase 4，默认 false = 与 Phase 1~3 逐字节相同】视觉 mesh 用哪一档。
-       true  = 复用 Phase 1 已经生成并入库的**抽稀件** `meshes/generated/<link>_collision.stl`
-               （VTK quadric decimation：base_link 2,078,226 → 3,000 面、l11 176,459 → 1,200 面；
-                bbox 与原件差 ≤3 mm，单位/原点不变 ⇒ 米制与几何位置都不改）。
-       false = 上游原始 STL（`meshes/<link>.STL`，base_link 那份 99 MiB / 207.8 万面）。
-       为什么需要：用户 2026-10-07 带 GUI 跑 robot:=robot11 时 **gzclient 被 SIGKILL（exit -9）**、
-       rviz2 黑屏 —— 就是这一档的渲染/内存代价（docs/robot_models.md §12 有实测对照）。
-       ⚠️ 只换 `<visual>`：`<collision>`（76 box + 云台细盒 + cylinder）一个字节都不动
-       ⇒ 物理/感知/契约完全不变；`robot:=robot11` 之外的模型根本不引用这两个 property。 -->
-  <xacro:arg name="visual_decimated" default="false"/>
+  <!-- ==========================================================================
+       【我们加的｜Phase 5（2026-10-07）】`<visual>` 用哪一档 mesh —— **只改渲染代价，不改几何**
+       —————————————————————————————————————
+       `robot11_visual:=decimated`（**默认**）⇒ `package://robot11/meshes/decimated/<link>.stl`
+          = Phase 5 生成的**视觉 LOD**：二次误差边折叠（QEM）抽稀，每 link ≤ 50k 面；
+            整车 2821320 → **163995** 面（141.1 MB → 8.2 MB，降 94%）。
+            逐 mesh 的"包围盒差 / 单向表面误差 p99,max / 三视剪影 IoU / 边界边"全部量化入库：
+            `robot11_description/inventory/visual_decimation.json`
+            （生成 + 验证：`tools/scripts/regress/robot11_decimate_visuals.py`，一条命令可复算）。
+            几个大头：base_link 2078226→50000, l11 176458→39999, l4 91234→11998, l5 90250→12000。
+       `robot11_visual:=full` ⇒ 上游原始 STL（`meshes/<link>.STL`；`base_link.STL` 99 MiB /
+          2,078,226 面）—— **只用于 A/B 对照**：带 GUI 跑就是这一档把 `gzclient` 撑到被内核
+          SIGKILL（exit -9）、`rviz2` 黑屏的（docs/robot_models.md §12 的实测表）。
+       为什么必须换（标准做法，引用见 docs/robot_models.md §13.2）：Gazebo Classic 的 `gzclient`
+       会把每个 `<visual>` 网格整份塞进渲染器；CAD 导出件（这里是整车 2821320 面）是给
+       "看/加工"用的，不是给"每帧渲染"用的。标准管线 = **视觉件与碰撞件分开** +
+       视觉件按每 link ≤ 50k 面（另一档公开口径是 ≤100k）抽稀 + 碰撞件用基本体/凸分解。
+       ⚠️ `<collision>`（carved（A 方案：DP box 减雷达视锥）、轮 cylinder、其余解析 box）与 `<inertial>`
+          **一个字节都不动** ⇒ 物理/感知/契约/质量/惯量完全不变。
+       ⚠️ 本段只被 `robot:=robot11` 引用 ⇒ 默认模型/其它槽位逐字节不变。 -->
+  <xacro:arg name="robot11_visual" default="decimated"/>
+  <xacro:arg name="visual_decimated" default=""/>
+  <xacro:property name="robot11_visual_p" value="$(arg robot11_visual)"/>
   <xacro:property name="visual_decimated_p" value="$(arg visual_decimated)"/>
-  <!-- ⚠️ xacro 会把 `"true"` 这个 arg **转成 Python 的 bool True**（实测：`${vd_p}` 打印 True），
-       所以这里必须 `str(...).lower()` 归一化，不能直接和字符串 'true' 比。 -->
-  <xacro:property name="visual_dir"
-      value="${'generated' if str(visual_decimated_p).lower() in ('true', '1') else 'meshes'}"/>
-  <xacro:property name="visual_ext"
-      value="${'_collision.stl' if str(visual_decimated_p).lower() in ('true', '1') else '.STL'}"/>
+  <!-- ⚠️ xacro 会把 `"true"` 这种 arg 转成 **Python bool**（实测 `${vd}` 打出 True）
+       ⇒ 必须 `str(...).lower()` 归一化后再比，不能直接和字符串 'true' 比。 -->
+  <xacro:property name="vd_norm" value="${str(visual_decimated_p).strip().lower()}"/>
+  <xacro:property name="rv_norm" value="${str(robot11_visual_p).strip().lower()}"/>
+  <xacro:property name="visual_full"
+      value="${(vd_norm in ('false', '0', 'no')) if vd_norm != '' else (rv_norm != 'decimated')}"/>
+  <xacro:property name="visual_dir" value="${'meshes' if visual_full else 'meshes/decimated'}"/>
+  <xacro:property name="visual_ext" value="${'.STL' if visual_full else '.stl'}"/>
   <!-- 【我们加的｜改名】上游根 link `body` → `base_link`（原因见文件头第 3 条）：
        本栈契约帧名是 base_link；不改名的实测后果 = TF 断树、LIO 发不出 /odom、
@@ -106,5 +130,5 @@
       <inertia ixx="0.012450840516849" ixy="8.34803982990868E-06" ixz="2.47736216819592E-06" iyy="0.0180415546421503" iyz="6.50018190294825E-06" izz="0.0214898895578463"/>
     </inertial>
-    <!-- 【上游原样】visual（**原始 mesh，视觉零损失**） -->
+    <!-- 【上游原样】visual（几何位置/单位/材质逐字照抄；mesh 文件按 `visual_dir` 换档，见文件头 Phase 5） -->
     <visual>
       <origin xyz="0 0 0" rpy="0 0 0"/>
@@ -434,5 +458,5 @@
       <inertia ixx="9.38551187090929E-05" ixy="-3.89659064263769E-08" ixz="-4.1188007722221E-07" iyy="0.000108022676479579" iyz="6.52751789180565E-07" izz="9.89453938308141E-05"/>
     </inertial>
-    <!-- 【上游原样】visual（**原始 mesh，视觉零损失**） -->
+    <!-- 【上游原样】visual（几何位置/单位/材质逐字照抄；mesh 文件按 `visual_dir` 换档，见文件头 Phase 5） -->
     <visual>
       <origin xyz="0 0 0" rpy="0 0 0"/>
@@ -455,5 +479,5 @@
       <inertia ixx="0.00027895263582235" ixy="4.01635255414384E-11" ixz="-1.35108698277116E-10" iyy="0.000144586311352007" iyz="4.08768977179887E-08" izz="0.000144975173531681"/>
     </inertial>
-    <!-- 【上游原样】visual（**原始 mesh，视觉零损失**） -->
+    <!-- 【上游原样】visual（几何位置/单位/材质逐字照抄；mesh 文件按 `visual_dir` 换档，见文件头 Phase 5） -->
     <visual>
       <origin xyz="0 0 0" rpy="0 0 0"/>
@@ -476,5 +500,5 @@
       <inertia ixx="9.38312233563086E-05" ixy="4.11880077230659E-07" ixz="-3.89659072508048E-08" iyy="9.87577896218705E-05" iyz="-6.52751787883143E-07" izz="0.00010783561712015"/>
     </inertial>
-    <!-- 【上游原样】visual（**原始 mesh，视觉零损失**） -->
+    <!-- 【上游原样】visual（几何位置/单位/材质逐字照抄；mesh 文件按 `visual_dir` 换档，见文件头 Phase 5） -->
     <visual>
       <origin xyz="0 0 0" rpy="0 0 0"/>
@@ -497,5 +521,5 @@
       <inertia ixx="0.000283619688479151" ixy="4.01635256040596E-11" ixz="-1.35108698263563E-10" iyy="0.000146944991593877" iyz="4.0876897717852E-08" izz="0.00014733385377355"/>
     </inertial>
-    <!-- 【上游原样】visual（**原始 mesh，视觉零损失**） -->
+    <!-- 【上游原样】visual（几何位置/单位/材质逐字照抄；mesh 文件按 `visual_dir` 换档，见文件头 Phase 5） -->
     <visual>
       <origin xyz="0 0 0" rpy="0 0 0"/>
@@ -518,5 +542,5 @@
       <inertia ixx="9.77808326150043E-05" ixy="3.89659073115738E-08" ixz="4.11880076872962E-07" iyy="0.000115206733276597" iyz="8.71786533446865E-07" izz="0.000102885906115304"/>
     </inertial>
-    <!-- 【上游原样】visual（**原始 mesh，视觉零损失**） -->
+    <!-- 【上游原样】visual（几何位置/单位/材质逐字照抄；mesh 文件按 `visual_dir` 换档，见文件头 Phase 5） -->
     <visual>
       <origin xyz="0 0 0" rpy="0 0 0"/>
@@ -539,5 +563,5 @@
       <inertia ixx="0.000283619688507033" ixy="4.01627190513287E-11" ixz="-1.35103941451045E-10" iyy="0.000146944991623376" iyz="4.08769024931138E-08" izz="0.000147333853773518"/>
     </inertial>
-    <!-- 【上游原样】visual（**原始 mesh，视觉零损失**） -->
+    <!-- 【上游原样】visual（几何位置/单位/材质逐字照抄；mesh 文件按 `visual_dir` 换档，见文件头 Phase 5） -->
     <visual>
       <origin xyz="0 0 0" rpy="0 0 0"/>
@@ -560,5 +584,5 @@
       <inertia ixx="9.72362930691966E-05" ixy="-4.11880085194013E-07" ixz="3.89659437807715E-08" iyy="0.000102339058097997" iyz="-8.3745233829181E-07" izz="0.000114151537565015"/>
     </inertial>
-    <!-- 【上游原样】visual（**原始 mesh，视觉零损失**） -->
+    <!-- 【上游原样】visual（几何位置/单位/材质逐字照抄；mesh 文件按 `visual_dir` 换档，见文件头 Phase 5） -->
     <visual>
       <origin xyz="0 0 0" rpy="0 0 0"/>
@@ -581,5 +605,5 @@
       <inertia ixx="0.000283619688507032" ixy="4.01627190942481E-11" ixz="-1.35103941448504E-10" iyy="0.000146944991623376" iyz="4.08769024930526E-08" izz="0.000147333853773518"/>
     </inertial>
-    <!-- 【上游原样】visual（**原始 mesh，视觉零损失**） -->
+    <!-- 【上游原样】visual（几何位置/单位/材质逐字照抄；mesh 文件按 `visual_dir` 换档，见文件头 Phase 5） -->
     <visual>
       <origin xyz="0 0 0" rpy="0 0 0"/>
@@ -602,5 +626,5 @@
       <inertia ixx="3.8779406325307E-05" ixy="1.66227406397812E-06" ixz="-3.65320210838414E-06" iyy="0.000141699871508992" iyz="-1.82170051595229E-11" izz="0.000141520295602471"/>
     </inertial>
-    <!-- 【上游原样】visual（**原始 mesh，视觉零损失**） -->
+    <!-- 【上游原样】visual（几何位置/单位/材质逐字照抄；mesh 文件按 `visual_dir` 换档，见文件头 Phase 5） -->
     <visual>
       <origin xyz="0 0 0" rpy="0 0 0"/>
@@ -649,5 +673,5 @@
       <inertia ixx="0.000577863329904443" ixy="-1.28185778246335E-07" ixz="3.64314989996771E-07" iyy="0.00058773469511404" iyz="-3.89011863670918E-05" izz="0.00023266714750829"/>
     </inertial>
-    <!-- 【上游原样】visual（**原始 mesh，视觉零损失**） -->
+    <!-- 【上游原样】visual（几何位置/单位/材质逐字照抄；mesh 文件按 `visual_dir` 换档，见文件头 Phase 5） -->
     <visual>
       <origin xyz="0 0 0" rpy="0 0 0"/>
@@ -756,5 +780,5 @@
       <inertia ixx="4.17032187760686E-05" ixy="-5.98077892665089E-09" ixz="3.05517185056836E-07" iyy="4.50191700802289E-05" iyz="-5.90930308926011E-10" izz="6.87178468496533E-05"/>
     </inertial>
-    <!-- 【上游原样】visual（**原始 mesh，视觉零损失**） -->
+    <!-- 【上游原样】visual（几何位置/单位/材质逐字照抄；mesh 文件按 `visual_dir` 换档，见文件头 Phase 5） -->
     <visual>
       <origin xyz="0 0 0" rpy="0 0 0"/>
