Commit message: fix(robot11): 底盘塌成单刚体 —— planar_move 的 Set*Vel 只对单刚体自洽，角速度通道 1.03%→16.2%
§L 把"robot11 几乎不执行角速度指令"登记为独立缺陷（§L.5/§L.9 第 2/3 项）但没钉死机理。本节钉死：

机理（源码级，gazebo/physics/Model.cc:746-771）：libgazebo_ros_planar_move.so 每次
OnUpdate 调 Model::SetLinearVel/SetAngularVel，而这两个函数是**把同一个 (v,ω) 写给模型里
每一个 link**。纯自转时它给每个 link 写 v=0、ω=(0,0,wz) —— 只有"整个模型是一个刚体、且绕
自身质心转"时才自洽；13 link / 12 joint 的 robot11 不自洽（第 i 个 link 的质心速度本应是
ω×r_i）⇒ 关节约束求解器每步把它掰回来，反作用吃掉底盘角速度。

台架判决（只发 /cmd_vel_chassis wz=1.0 × 12 仿真秒 = 请求 687.5°，同一世界/出生点）：
  · robot11 原样         +7.09°（1.03%）       · 单刚体（本修法）  +111.7…113.3°（16.2~16.5%）
  · 全关节改 fixed       +21.31°（3.10%）      · 默认模型（对照）  +40.01°（5.82%）
  · 零重力/无接触        +128.02°（18.6%）     · 极简单 link box   +681.25°（99.9%）
自由偏航漂移（无指令 60 s）：+18.4° → +0.02°（默认模型 −0.24°）。
盲推正前方被实体障碍挡住的极限不变：0.4077 → 0.3998 m（§L 记 0.4199 m）。

做法（只动"哪条 link 装哪块几何"，不动任何一块几何、不动总质量/惯量）：
  · l2…l11 的 collision/visual pose 经 FK 变换到根 link 后逐条挂过来；
  · 惯量按平行轴定理合成（M=9.4121 kg、Izz=0.126766 kg·m²）；
  · 删 j2…j11，**保留** livox_frame / imu_link 及其固定关节（感知链的帧与传感器不动）；
  · 自证不通过就不生成：碰撞 AABB 逐条相等 + 整车最低点必须落在轮子上（−0.10250 m）。
    第二条实际救过一次 —— 自证只比"塌陷前后"，FK 静默退化（rpy 被按 6 个数解析读成零向量）
    时两边会一起错、照样通过；"最低点在轮上"这条不依赖 FK 正确性。

回退：robot11_make_sim_xacro.py --chassis articulated（输出与 HEAD 逐字节相同，已核 sha256）。

实测数字、逐候选判决表、被否掉的修法（update_rate=1000：角速度 7.8% 但盲推能爬上障碍
2.57 m / z 0.15→0.40，且不解决漂移）、新验收口径见下两个 commit 与
docs/tilted_lidar_fidelity.md §M。

File: src/rm_nav_bringup/urdf/sentry_robot_robot11_sim.xacro (robot description, xacro)
@@ -1,90 +1,21 @@
 <?xml version="1.0"?>
-<!--
-  ============================================================================
-  sentry_robot_robot11_sim.xacro —— `robot:=robot11` 槽位的机器人模型（**opt-in，不是默认**）
-  ============================================================================
-  ⚠️ **本文件是生成的，不要手改**：由
-       tools/scripts/regress/robot11_make_sim_xacro.py
-     从上游 `urdf/upstream/robot11.urdf`（sha256 e3e322acbe06996fc8adf410af5c0fcab7207de6cb76bf7234310bab2b3a64fc）+ Phase 1 的碰撞清单
-     `robot11_description/inventory/collision_assets.json` 生成。
-     改生成器 → 重跑 → 提交；手改会在下次重跑时被覆盖。
-  ── 上游来源（用户 2026-10-07 在会话里贴出，另一个 agent 逐字重建） ──────────
-    文件：`.tmp_urdf2/robot11.urdf`（11737 B）→ 本仓逐字节副本
-          `src/rm_nav_bringup/urdf/upstream/robot11.urdf`（**只读、不参与运行**，仅供核对）
-    sha256：e3e322acbe06996fc8adf410af5c0fcab7207de6cb76bf7234310bab2b3a64fc
-    根 link：`body`；12 个 link / 12 个 joint；机器人名 `sentry`
-    它**自带** `<inertial>`（与 hzmirm 那份不同）⇒ 不需要我们补惯性
-    mesh：`package://robot11/meshes/<name>.STL`（**这正是"包名必须叫 robot11"的原因**）
-  ── 上游自相矛盾的一处（本文件用 arg 留了开关，不猜） ──────────────────────
-    `body_to_livox` 的 30° 旋转轴：
-      · URDF 原文写 `rpy="0 -0.5236 0"`（绕 y = pitch）
-      · 同一台车的 SolidWorks CSV 写 `Joint Origin Roll = -0.523598775598293`（绕 x = roll）
-    本文件默认按 **CSV 的 roll 形式**（机器导出的 CSV 比手打的一行更可能是字面真相），
-    但把它参数化成 `livox_tilt_rpy`，并给了 `livox_tilt_axis:=roll|pitch` 这个 launch 开关。
-    ⚠️ 几何事实（§9.5 已推过、Phase 2 实测复核）：MID-360 方位 360° ⇒ 两个候选的
-    **世界仰角谱与地面环半径完全相同**，只差一个绕 z 的旋转；**唯一判据是"最朝下的方位"**。
-  ── `【上游原样】/【我们加的】` 两种标记 ────────────────────────────────────
-    【上游原样】= 与上游 URDF 数值逐字相同（脚本生成，可重算）
-    【我们加的】= 本栈要跑起来必须补的（逐条写理由与日期）
-  ── Phase 3（2026-10-07）：让雷达"看得出去" + 斜置感知链 ─────────────────────
-    用户的判定（两条，都已按它执行）：
-      (1) **30° 是绕 roll**（用户按实物确认）⇒ 本文件的默认 `livox_tilt_rpy` = roll 形式；
-      (2) 上游 URDF/mesh "跟实物基本一致，仿真侧可以改" ⇒ 允许仿真侧适配，
-         但**每一处偏离都要写日期 + 中文理由 + provenance 表**（见 docs/robot_models.md §11）。
-    Phase 2 的结论是"这台车的雷达在底盘凹槽里，看不见外面"（75.5% 的点是自击、无 /odom）。
-    Phase 3 用**三种方案**实测（离线 30000 条射线 + Gazebo 无头跑）：
-      A（保真优先，**采用**）：body 碰撞 = DP box 减视锥（`—body-collision carved`）⇒ 雷达仍在
-         上游的 0.2595 m 高度，只把"凹槽开口"在碰撞里显式挖出来；
-      B（仿真适配）：保留 4 个 box，把 `livox_frame` 抬高（`—livox-raise-m`）⇒ 离线扫描：
-         +0.05 m 仍 96.6% 自击、+0.06 m 降到 19.8%、**+0.08 m 才干净（0.24%）**、
-         +0.10 m 起与 A 等价（0% 自击 / 25.2% 看见地面）—— 代价是雷达离地 0.2595 → 0.3595 m，
-         与本仓默认模型的 0.226 m 差得更远，且 linefit 的 sensor_height 必须跟着变；
-      C（抽稀网格碰撞）：**已查清**：spawn 正常但传感器一条数据都没有 —— 根因是 ODE 的
-         ray-vs-trimesh 是 O(#三角面) 的，30000 条射线 × 3000 面 = 9×10⁷ 次/帧 @10 Hz
-         ⇒ gzserver 在"打一帧射线"里出不来（传感器回调永不返回），不是插件没挂上。
-    倾斜感知链（**全部只对本槽位生效**，默认模型逐字节不变）：
-      · linefit：`sensor_height` = 雷达离地（0.2595 + raise）、`gravity_aligned_frame` = base_link
-        （雷达斜 30° ⇒ 传感器系的 z 不再是"高度"）—— 见 `config/segmentation_sim_robot11.yaml`
-      · pointcloud_to_laserscan：`target_frame` = base_link（高度带改在重力对齐系里量）
-        —— 见 `config/laserscan_params_robot11.yaml`
-      · LIO 外参：**不改**。IMU 与雷达同壳、只差 0.05 m 平移（`extrinsic_T=[0,0,0.05]`,
-        `extrinsic_R=I` 逐字节沿用），IMU 姿态里的 30° 由 LIO 自己估出来，
-        `odom→base_link` 由 small_point_lio 用 `base_link→livox_frame` 的 TF 精确换算。
-  ── ⚠️ 上游的 <collision> 全被替换掉了（这是本槽位最关键的一处偏离） ────────
-    上游 12 个 link 的 collision **全部是 mesh**，其中 `body` = 2,078,226 面。
-    Phase 1 实测（极简世界单模型 spawn，无头隔离，见 docs/robot_models.md §9.3）：
-      · 稳态悬空 RTF 1.002（没有接触对 ⇒ 别拿这个当"能用"）
-      · **一有接触** RTF **0.200**、最低 0.04（慢 25–50 倍）；同工况 4 个 box = 1.002
-      · 峰值内存恒 **759 MB vs 基线 172 MB**
-    ⇒ 替换为：`body` = 4 个 box（DP 最优分段包络，覆盖率 1.000、总体积只比凸包胖 9.4%）；
-      轮 = cylinder；其余 = 抽稀件。
-  ── Phase 5（2026-10-07）：把 `<visual>` 也换档（**这才是"带 GUI 放得进仿真"的那一步**）──
-    Phase 1~3 只改了**碰撞**侧，**视觉**侧一直是上游原始 STL：整车 **2,821,320 面 / 141.07 MB**
-    `base_link.STL` 一项 2,078,226 面 / 99 MiB。用户 2026-10-07 带 GUI 跑 ⇒ **gzclient 被内核
-    SIGKILL（exit -9）**、rviz2 黑屏 —— 因为 gzclient 会把每个 `<visual>` 网格整份渲进 OGRE。
-    Phase 5 按公开的标准管线（视觉/碰撞分离 + QEM 抽稀 + 量化验证，引用见 docs/robot_models.md
-    §13.2）生成**视觉 LOD**：每 link ≤ 50k 面、整车 ≤ 200k 面，逐 mesh 量化"包围盒差 /
-    单向表面误差 p99,max / 三视剪影 IoU / 边界边数"，全部落在
-    `robot11_description/inventory/visual_decimation.json`。
-    开关：`robot11_visual:=decimated`（**默认**）| `full`；`<collision>` 与 `<inertial>` 不动。
--->
-<robot name="sentry" xmlns:xacro="http://ros.org/wiki/xacro">
+<robot xmlns:xacro="http://ros.org/wiki/xacro" name="sentry">
   <!-- 【我们加的】launch 会无条件传平台外参（bringup_sim.launch.py 的 xyz/rpy）。
        本模型的雷达位姿由上游关节链唯一决定 ⇒ 这两个参数**声明但不用**（与 hzmirm 槽位同款理由：
        再叠一个外部平移就等于改上游几何）。 -->
-  <xacro:arg name="xyz" default="0 0 0"/>
-  <xacro:arg name="rpy" default="0 0 0"/>
+  <xacro:arg name="xyz" default="0 0 0" />
+  <xacro:arg name="rpy" default="0 0 0" />
   <!-- 【我们加的】雷达 30° 安装的旋转；默认 = SolidWorks CSV 的 roll 形式
        （用户 2026-10-07 **按实物确认：是绕 roll**；pitch 只作对照开关）。
        pitch 形式 = "0 -0.523598775598293 0"。两者对 360° 雷达几何等价（差一个绕 z 的旋转）。 -->
-  <xacro:arg name="livox_tilt_rpy" default="-0.523598775598293 0 0"/>
+  <xacro:arg name="livox_tilt_rpy" default="-0.523598775598293 0 0" />
   <!-- 【我们加的｜B 方案，默认 0 = 与上游逐字相同】把雷达（连同 IMU）整体抬高的米数。
        用途：实测"不做碰撞开口、直接把雷达抬到顶板上方"这条仿真适配路（docs/robot_models.md §11）。
        ⚠️ 抬高会改变雷达离地高度 ⇒ linefit 的 sensor_height 必须同步 = 0.2595 + livox_raise_m
        （launch 里由 robot:=robot11 分支**算出来**注入，不是手抄）。默认 0 ⇒ 一切不变。 -->
-  <xacro:arg name="livox_raise_m" default="0"/>
+  <xacro:arg name="livox_raise_m" default="0" />
   <!-- xacro 的表达式里**不能直接写 arg 名**（实测报 name 'livox_raise_m' is not defined）
        ⇒ 按标准写法先绑成 property 再进表达式。 -->
-  <xacro:property name="livox_raise_m_p" value="$(arg livox_raise_m)"/>
+  <xacro:property name="livox_raise_m_p" value="$(arg livox_raise_m)" />
   <!-- ==========================================================================
        【我们加的｜2026-10-08，2026-10-09 扩展第三档】**雷达安装方式**开关
@@ -117,18 +48,15 @@
        `<cloud_frame>` 元素；它的两处 property 取值与 urdf 档完全相同）—— 见 §J 的静态证据。
        ========================================================================== -->
-  <xacro:arg name="livox_mount" default="plugin"/>
-  <xacro:property name="livox_mount_p" value="$(arg livox_mount)"/>
-  <xacro:property name="livox_tilt_rpy_p" value="$(arg livox_tilt_rpy)"/>
+  <xacro:arg name="livox_mount" default="plugin" />
+  <xacro:property name="livox_mount_p" value="$(arg livox_mount)" />
+  <xacro:property name="livox_tilt_rpy_p" value="$(arg livox_tilt_rpy)" />
   <!-- 倾角记在**关节**上的两档（urdf / sensor）：关节 rpy = 倾角、插件 <tilt_rpy> = 单位阵 -->
-  <xacro:property name="livox_mount_tilt_in_joint"
-                  value="${livox_mount_p.strip() in ('urdf', 'sensor')}"/>
+  <xacro:property name="livox_mount_tilt_in_joint" value="${livox_mount_p.strip() in ('urdf', 'sensor')}" />
   <!-- 点云表达在**传感器系**的那一档（sensor；缺省/plugin/urdf = 父 link 系） -->
-  <xacro:property name="livox_mount_sensor" value="${livox_mount_p.strip() == 'sensor'}"/>
+  <xacro:property name="livox_mount_sensor" value="${livox_mount_p.strip() == 'sensor'}" />
   <!-- 关节 rpy：urdf/sensor 档 = 倾角；plugin 档 = 0 -->
-  <xacro:property name="livox_joint_rpy"
-                  value="${livox_tilt_rpy_p if livox_mount_tilt_in_joint else '0 0 0'}"/>
+  <xacro:property name="livox_joint_rpy" value="${livox_tilt_rpy_p if livox_mount_tilt_in_joint else '0 0 0'}" />
   <!-- 插件 <tilt_rpy>：plugin 档 = 倾角；urdf/sensor 档 = 单位阵（射线已由 link 姿态带斜） -->
-  <xacro:property name="livox_plugin_tilt_rpy"
-                  value="${'0 0 0' if livox_mount_tilt_in_joint else livox_tilt_rpy_p}"/>
+  <xacro:property name="livox_plugin_tilt_rpy" value="${'0 0 0' if livox_mount_tilt_in_joint else livox_tilt_rpy_p}" />
   <!-- ==========================================================================
        【我们加的｜Phase 5（2026-10-07）】`<visual>` 用哪一档 mesh —— **只改渲染代价，不改几何**
@@ -151,16 +79,15 @@
           **一个字节都不动** ⇒ 物理/感知/契约/质量/惯量完全不变。
        ⚠️ 本段只被 `robot:=robot11` 引用 ⇒ 默认模型/其它槽位逐字节不变。 -->
-  <xacro:arg name="robot11_visual" default="decimated"/>
-  <xacro:arg name="visual_decimated" default=""/>
-  <xacro:property name="robot11_visual_p" value="$(arg robot11_visual)"/>
-  <xacro:property name="visual_decimated_p" value="$(arg visual_decimated)"/>
+  <xacro:arg name="robot11_visual" default="decimated" />
+  <xacro:arg name="visual_decimated" default="" />
+  <xacro:property name="robot11_visual_p" value="$(arg robot11_visual)" />
+  <xacro:property name="visual_decimated_p" value="$(arg visual_decimated)" />
   <!-- ⚠️ xacro 会把 `"true"` 这种 arg 转成 **Python bool**（实测 `${vd}` 打出 True）
        ⇒ 必须 `str(...).lower()` 归一化后再比，不能直接和字符串 'true' 比。 -->
-  <xacro:property name="vd_norm" value="${str(visual_decimated_p).strip().lower()}"/>
-  <xacro:property name="rv_norm" value="${str(robot11_visual_p).strip().lower()}"/>
-  <xacro:property name="visual_full"
-      value="${(vd_norm in ('false', '0', 'no')) if vd_norm != '' else (rv_norm != 'decimated')}"/>
-  <xacro:property name="visual_dir" value="${'meshes' if visual_full else 'meshes/decimated'}"/>
-  <xacro:property name="visual_ext" value="${'.STL' if visual_full else '.stl'}"/>
+  <xacro:property name="vd_norm" value="${str(visual_decimated_p).strip().lower()}" />
+  <xacro:property name="rv_norm" value="${str(robot11_visual_p).strip().lower()}" />
+  <xacro:property name="visual_full" value="${(vd_norm in ('false', '0', 'no')) if vd_norm != '' else (rv_norm != 'decimated')}" />
+  <xacro:property name="visual_dir" value="${'meshes' if visual_full else 'meshes/decimated'}" />
+  <xacro:property name="visual_ext" value="${'.STL' if visual_full else '.stl'}" />
   <!-- 【我们加的｜改名】上游根 link `body` → `base_link`（原因见文件头第 3 条）：
        本栈契约帧名是 base_link；不改名的实测后果 = TF 断树、LIO 发不出 /odom、
@@ -168,15 +95,10 @@
   <!-- ==================== link base_link ==================== -->
   <link name="base_link">
-    <!-- 【上游原样】inertial -->
-    <inertial>
-      <origin xyz="0.00436933539925447 0.0121729882941287 0.0624624952683773" rpy="0 0 0"/>
-      <mass value="6.98390841611154"/>
-      <inertia ixx="0.012450840516849" ixy="8.34803982990868E-06" ixz="2.47736216819592E-06" iyy="0.0180415546421503" iyz="6.50018190294825E-06" izz="0.0214898895578463"/>
-    </inertial>
+    <inertial><origin xyz="0.00355133581 0.00712115226 0.0731223016" rpy="0 0 0" /><mass value="9.41213494" /><inertia ixx="0.14791895" ixy="-0.000219710256" ixz="0.000492592844" iyy="0.151973674" iyz="0.00854664536" izz="0.126766291" /></inertial><!-- 【上游原样】inertial -->
     <!-- 【上游原样】visual（几何位置/单位/材质逐字照抄；mesh 文件按 `visual_dir` 换档，见文件头 Phase 5） -->
     <visual>
-      <origin xyz="0 0 0" rpy="0 0 0"/>
-      <geometry><mesh filename="package://robot11/${visual_dir}/base_link${visual_ext}"/></geometry>
-      <material name=""><color rgba="0.792156862745098 0.819607843137255 0.933333333333333 1"/></material>
+      <origin xyz="0 0 0" rpy="0 0 0" />
+      <geometry><mesh filename="package://robot11/${visual_dir}/base_link${visual_ext}" /></geometry>
+      <material name=""><color rgba="0.792156862745098 0.819607843137255 0.933333333333333 1" /></material>
     </visual>
     <!-- 【我们加的｜替换】上游这里是 mesh collision；按 Phase 1 实测换掉（原因见文件头） -->
@@ -190,643 +112,529 @@
          ⚠️ 这是**仿真侧适配**（偏离上游 CAD 的碰撞几何），逐条登记在 docs/robot_models.md §11 -->
     <collision>
-      <origin xyz="0.000000 0.000000 -0.040269" rpy="0 0 0"/>
-      <geometry><box size="0.600000 0.600000 0.015350"/></geometry>
-    </collision>
-    <collision>
-      <origin xyz="0.000000 -0.007500 -0.024920" rpy="0 0 0"/>
-      <geometry><box size="0.600000 0.585000 0.015350"/></geometry>
-    </collision>
-    <collision>
-      <origin xyz="0.000000 -0.015000 -0.009570" rpy="0 0 0"/>
-      <geometry><box size="0.600000 0.570000 0.015350"/></geometry>
-    </collision>
-    <collision>
-      <origin xyz="0.000000 -0.030000 0.005780" rpy="0 0 0"/>
-      <geometry><box size="0.600000 0.540000 0.015350"/></geometry>
-    </collision>
-    <collision>
-      <origin xyz="0.000000 -0.037500 0.021129" rpy="0 0 0"/>
-      <geometry><box size="0.600000 0.525000 0.015350"/></geometry>
-    </collision>
-    <collision>
-      <origin xyz="0.000000 -0.052500 0.036479" rpy="0 0 0"/>
-      <geometry><box size="0.600000 0.495000 0.015350"/></geometry>
-    </collision>
-    <collision>
-      <origin xyz="0.000000 -0.037500 0.051829" rpy="0 0 0"/>
-      <geometry><box size="0.540000 0.465000 0.015350"/></geometry>
-    </collision>
-    <collision>
-      <origin xyz="0.000000 -0.052500 0.067178" rpy="0 0 0"/>
-      <geometry><box size="0.540000 0.435000 0.015350"/></geometry>
-    </collision>
-    <collision>
-      <origin xyz="0.000000 -0.067500 0.082528" rpy="0 0 0"/>
-      <geometry><box size="0.540000 0.405000 0.015350"/></geometry>
-    </collision>
-    <collision>
-      <origin xyz="0.000000 -0.075000 0.097878" rpy="0 0 0"/>
-      <geometry><box size="0.540000 0.390000 0.015350"/></geometry>
-    </collision>
-    <collision>
-      <origin xyz="0.000000 -0.045000 0.113227" rpy="0 0 0"/>
-      <geometry><box size="0.540000 0.270000 0.015350"/></geometry>
-    </collision>
-    <collision>
-      <origin xyz="0.000000 -0.060000 0.128577" rpy="0 0 0"/>
-      <geometry><box size="0.540000 0.240000 0.015350"/></geometry>
-    </collision>
-    <collision>
-      <origin xyz="0.000000 -0.060000 0.143927" rpy="0 0 0"/>
-      <geometry><box size="0.300000 0.270000 0.015350"/></geometry>
-    </collision>
-    <collision>
-      <origin xyz="0.000000 -0.075000 0.159276" rpy="0 0 0"/>
-      <geometry><box size="0.300000 0.240000 0.015350"/></geometry>
-    </collision>
-    <collision>
-      <origin xyz="0.000000 -0.090000 0.174626" rpy="0 0 0"/>
-      <geometry><box size="0.300000 0.210000 0.015350"/></geometry>
-    </collision>
-    <collision>
-      <origin xyz="0.000000 -0.112500 0.189976" rpy="0 0 0"/>
-      <geometry><box size="0.300000 0.165000 0.015350"/></geometry>
-    </collision>
-    <collision>
-      <origin xyz="0.000000 -0.127500 0.205325" rpy="0 0 0"/>
-      <geometry><box size="0.300000 0.135000 0.015350"/></geometry>
-    </collision>
-    <collision>
-      <origin xyz="0.000000 0.247500 0.005780" rpy="0 0 0"/>
-      <geometry><box size="0.570000 0.015000 0.015350"/></geometry>
-    </collision>
-    <collision>
-      <origin xyz="0.000000 0.202500 0.036479" rpy="0 0 0"/>
-      <geometry><box size="0.570000 0.015000 0.015350"/></geometry>
-    </collision>
-    <collision>
-      <origin xyz="0.007500 0.292500 -0.024920" rpy="0 0 0"/>
-      <geometry><box size="0.555000 0.015000 0.015350"/></geometry>
-    </collision>
-    <collision>
-      <origin xyz="0.007500 0.232500 0.021129" rpy="0 0 0"/>
-      <geometry><box size="0.525000 0.015000 0.015350"/></geometry>
-    </collision>
-    <collision>
-      <origin xyz="0.000000 0.277500 -0.009570" rpy="0 0 0"/>
-      <geometry><box size="0.510000 0.015000 0.015350"/></geometry>
-    </collision>
-    <collision>
-      <origin xyz="0.000000 0.142500 0.082528" rpy="0 0 0"/>
-      <geometry><box size="0.510000 0.015000 0.015350"/></geometry>
-    </collision>
-    <collision>
-      <origin xyz="0.000000 0.217500 0.036479" rpy="0 0 0"/>
-      <geometry><box size="0.480000 0.015000 0.015350"/></geometry>
-    </collision>
-    <collision>
-      <origin xyz="0.000000 0.172500 0.067178" rpy="0 0 0"/>
-      <geometry><box size="0.480000 0.015000 0.015350"/></geometry>
-    </collision>
-    <collision>
-      <origin xyz="0.000000 0.097500 0.113227" rpy="0 0 0"/>
-      <geometry><box size="0.480000 0.015000 0.015350"/></geometry>
-    </collision>
-    <collision>
-      <origin xyz="0.000000 0.067500 0.128577" rpy="0 0 0"/>
-      <geometry><box size="0.480000 0.015000 0.015350"/></geometry>
-    </collision>
-    <collision>
-      <origin xyz="0.000000 0.262500 0.005780" rpy="0 0 0"/>
-      <geometry><box size="0.450000 0.015000 0.015350"/></geometry>
-    </collision>
-    <collision>
-      <origin xyz="0.000000 0.127500 0.097878" rpy="0 0 0"/>
-      <geometry><box size="0.450000 0.015000 0.015350"/></geometry>
-    </collision>
-    <collision>
-      <origin xyz="0.000000 0.247500 0.021129" rpy="0 0 0"/>
-      <geometry><box size="0.420000 0.015000 0.015350"/></geometry>
-    </collision>
-    <collision>
-      <origin xyz="0.000000 0.202500 0.051829" rpy="0 0 0"/>
-      <geometry><box size="0.420000 0.015000 0.015350"/></geometry>
-    </collision>
-    <collision>
-      <origin xyz="0.000000 0.157500 0.082528" rpy="0 0 0"/>
-      <geometry><box size="0.420000 0.015000 0.015350"/></geometry>
-    </collision>
-    <collision>
-      <origin xyz="0.000000 0.082500 0.128577" rpy="0 0 0"/>
-      <geometry><box size="0.420000 0.015000 0.015350"/></geometry>
-    </collision>
-    <collision>
-      <origin xyz="0.000000 0.292500 -0.009570" rpy="0 0 0"/>
-      <geometry><box size="0.360000 0.015000 0.015350"/></geometry>
-    </collision>
-    <collision>
-      <origin xyz="0.000000 0.232500 0.036479" rpy="0 0 0"/>
-      <geometry><box size="0.360000 0.015000 0.015350"/></geometry>
-    </collision>
-    <collision>
-      <origin xyz="0.000000 0.187500 0.067178" rpy="0 0 0"/>
-      <geometry><box size="0.360000 0.015000 0.015350"/></geometry>
-    </collision>
-    <collision>
-      <origin xyz="0.000000 0.142500 0.097878" rpy="0 0 0"/>
-      <geometry><box size="0.360000 0.015000 0.015350"/></geometry>
-    </collision>
-    <collision>
-      <origin xyz="0.000000 0.172500 0.082528" rpy="0 0 0"/>
-      <geometry><box size="0.330000 0.015000 0.015350"/></geometry>
-    </collision>
-    <collision>
-      <origin xyz="0.000000 0.277500 0.005780" rpy="0 0 0"/>
-      <geometry><box size="0.300000 0.015000 0.015350"/></geometry>
-    </collision>
-    <collision>
-      <origin xyz="0.000000 0.217500 0.051829" rpy="0 0 0"/>
-      <geometry><box size="0.300000 0.015000 0.015350"/></geometry>
-    </collision>
-    <collision>
-      <origin xyz="0.007500 -0.022500 0.189976" rpy="0 0 0"/>
-      <geometry><box size="0.285000 0.015000 0.015350"/></geometry>
-    </collision>
-    <collision>
-      <origin xyz="0.000000 0.262500 0.021129" rpy="0 0 0"/>
-      <geometry><box size="0.270000 0.015000 0.015350"/></geometry>
-    </collision>
-    <collision>
-      <origin xyz="0.000000 0.202500 0.067178" rpy="0 0 0"/>
-      <geometry><box size="0.270000 0.015000 0.015350"/></geometry>
-    </collision>
-    <collision>
-      <origin xyz="0.000000 0.157500 0.097878" rpy="0 0 0"/>
-      <geometry><box size="0.270000 0.015000 0.015350"/></geometry>
-    </collision>
-    <collision>
-      <origin xyz="0.000000 0.082500 0.143927" rpy="0 0 0"/>
-      <geometry><box size="0.270000 0.015000 0.015350"/></geometry>
-    </collision>
-    <collision>
-      <origin xyz="0.000000 0.052500 0.159276" rpy="0 0 0"/>
-      <geometry><box size="0.240000 0.015000 0.015350"/></geometry>
-    </collision>
-    <collision>
-      <origin xyz="0.000000 0.022500 0.174626" rpy="0 0 0"/>
-      <geometry><box size="0.240000 0.015000 0.015350"/></geometry>
-    </collision>
-    <collision>
-      <origin xyz="0.000000 -0.052500 0.205325" rpy="0 0 0"/>
-      <geometry><box size="0.240000 0.015000 0.015350"/></geometry>
-    </collision>
-    <collision>
-      <origin xyz="0.000000 0.247500 0.036479" rpy="0 0 0"/>
-      <geometry><box size="0.210000 0.015000 0.015350"/></geometry>
-    </collision>
-    <collision>
-      <origin xyz="0.000000 0.187500 0.082528" rpy="0 0 0"/>
-      <geometry><box size="0.210000 0.015000 0.015350"/></geometry>
-    </collision>
-    <collision>
-      <origin xyz="-0.105000 0.112500 0.113227" rpy="0 0 0"/>
-      <geometry><box size="0.180000 0.015000 0.015350"/></geometry>
-    </collision>
-    <collision>
-      <origin xyz="0.105000 0.112500 0.113227" rpy="0 0 0"/>
-      <geometry><box size="0.180000 0.015000 0.015350"/></geometry>
-    </collision>
-    <collision>
-      <origin xyz="0.000000 0.067500 0.159276" rpy="0 0 0"/>
-      <geometry><box size="0.180000 0.015000 0.015350"/></geometry>
-    </collision>
-    <collision>
-      <origin xyz="0.000000 -0.007500 0.189976" rpy="0 0 0"/>
-      <geometry><box size="0.180000 0.015000 0.015350"/></geometry>
-    </collision>
-    <collision>
-      <origin xyz="0.000000 0.232500 0.051829" rpy="0 0 0"/>
-      <geometry><box size="0.150000 0.015000 0.015350"/></geometry>
-    </collision>
-    <collision>
-      <origin xyz="0.000000 0.172500 0.097878" rpy="0 0 0"/>
-      <geometry><box size="0.150000 0.015000 0.015350"/></geometry>
-    </collision>
-    <collision>
-      <origin xyz="0.000000 0.037500 0.174626" rpy="0 0 0"/>
-      <geometry><box size="0.150000 0.015000 0.015350"/></geometry>
-    </collision>
-    <collision>
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