Commit message: fix(sim): robot11 也真的能原地转 —— 单刚体早就有，缺的是轮子对地摩擦（10.6% → 95.8%）
实测缺陷（本机 Classic，真值 /odom_ground_truth + 仿真时间口径）：
  纯原地转 wz=0.8 → 台架 9.713°/91.7° = 10.6%；整栈 20 Hz 8.94°/2 s = 9.8%
  纯前进   vx=0.30 → 台架 79.3%；整栈 20 Hz 55.2%（"前进正常"其实也吃了 ~20%）
归因（aa77420 的两项里，robot11 只剩第二项）：
  ① 结构：已经满足 —— 2026-10-10 的 robot11_weld_chassis.py 早把 l2…l11 塌成一个刚体，
     gz sdf -p = 1 link / 0 joint / 113 collision（planar_move 的 Set*Vel 本来就自洽）；
  ② 摩擦：唯一剩下的 —— 改前 SDF 里 113 条 collision 的 <surface><friction><ode> **全是空的**
     （ODE 缺省 μ=1 ⇒ 4 个轮子横向刮地）；上游 robot11.urdf 里根本没有 mu1/mu2，生成器只搬
     inertial/visual/collision，塌陷时又删掉指向 l6…l9 的 <gazebo reference>；而 Gazebo 只认
     <gazebo reference>（写在 <link> 里的 mu1/mu2 会被忽略）。
修法（最小面：生成器 + 一个生成物；源文件一个字节没改）：
  · robot11_make_sim_xacro.py：新增 --wheel-mu（缺省 0.02）/ --no-wheel-friction；
    在 FOOTER 里写 <gazebo reference="base_link"><mu1>/<mu2>（轮子已塌进 base_link，没有
    wheel_N 可写）；写文件前用 gz sdf -p 自证：1 link、113 条 collision 的 friction 全部 = μ、
    4 条轮 cylinder、113 条碰撞 AABB 与 URDF 逐条相等（最大偏差 5e-6 m）、mass/Izz 与全 link
    平行轴定理合成值相等；不通过就不写文件。
  · 生成物 sentry_robot_robot11_sim.xacro 重新生成（相对 HEAD 只多摩擦块 + 两段注释；SDF 文本
    diff 只有 113 组 <ode/> → <ode><mu>0.02</mu><mu2>0.02</mu2></ode>）。
  · robot11_weld_chassis.py：weld(..., extra_note='') 把摩擦说明写进生成物末尾那段注释。
  · --no-wheel-friction 与 HEAD 逐字节相同；--chassis articulated 模型体去注释后逐字节相同，
    install/ 是逐文件符号链接 ⇒ 不需要 colcon build。launch/槽位/robot11_mount 一字未动。
实测（修后）：台架自转 95.8%、整栈 20 Hz 92.9% / 200 Hz 95.3%，前进 88.6%（台架）/ 98.2%（整栈）；
  剂量-响应 μ=0.2/0.1/0.05/0.02/0.001 → 66.9/82.3/89.6/95.8/98.3%。
  几何不变：1 link、113 条 AABB 逐条相等、轮 r=0.058 L=0.0452/0.0453 与中心不变、最低点
  −0.102502 m 在轮上、mass 9.56212 / Izz 0.129172 不变、body_to_livox 安装位姿逐字不变、h=0.259527。
  代价（故意改的物理）：静摩擦角 atan(0.02) ≈ 1.1° ⇒ 更陡的坡上停住会滑（速度驱动爬坡不受影响）；
  要更抓地就 --wheel-mu 0.1（≈82.3%、≈5.7° 坡）。盲推 25 s 仍停在 0.4000 m、z 不变（不爬障碍）。
下游冒烟：mode:=nav localization:=gicp robot:=robot11 robot11_mount:=sensor lio:=small_point_lio
  （gravity_align 自动 hybrid）2 跑：local costmap 非空（lethal 中位 342/327、最近 0.708/0.715 m）、
  h_meas 0.2616 m INFO、墙面残差 0.0000（插件修 7a544bf 仍成立）。
详见 docs/frame_contract_v3_measurements.md §22（含诚实清单：μ 是全 link 生效、坡未实测、
nav local lethal 高于 §21 参考带且未做改前 A/B 等）。

File: src/rm_nav_bringup/urdf/sentry_robot_robot11_sim.xacro (robot description, xacro)
@@ -836,4 +836,28 @@
   <gazebo reference="livox_frame"><material>Gazebo/LightBlueLaser</material></gazebo>
   <gazebo reference="imu_link"><material>Gazebo/BuildingFrame</material></gazebo>
+  <!-- ⑥ 【我们加的｜2026-10-20】**轮子对地摩擦**（★ Gazebo 只认 `<gazebo reference>` 这一种写法）
+       ———————————————————————————————————————
+       为什么（实测，见 docs/frame_contract_v3_measurements.md §22）：本模型被塌成**单个刚体**后，
+       轮子不能再靠滚动"让开"，原地转 = 4 个轮子同时**横向刮地** ⇒ 摩擦项直接吃掉角速度。
+       改前（Gazebo 缺省 μ=1，SDF 里 `surface/friction/ode` 是空的）：纯自转 wz=0.8 → **10.6%**（台架）/
+       **9.8%**（整栈 20 Hz）；纯前进 vx=0.3 → 79.3%（台架）/ 55.2%（整栈）。
+       加上 μ=0.02 后：台架自转 **95.8%**、整栈 20 Hz **92.9%** / 200 Hz **95.3%**（与默认模型 §20 同一条剂量-响应）。
+       ⚠️ 两个容易踩的坑，本文件都绕开了：
+         (a) `<mu1>/<mu2>` 写在 `<link>` **里面** = Gazebo 的 URDF 解析器**不认**（等于没写）；
+             必须写成 `<gazebo reference="<link>">`。`gz sdf -p` 之后每个 collision 都应真的出现
+             `<surface><friction><ode><mu>/<mu2>` 且等于这里给的值 —— 生成器每次都自证（不通过不写文件）。
+         (b) 轮子 `l6..l9` 已被 `robot11_weld_chassis.py` 塌进 base_link（它们不再是 link）
+             ⇒ 摩擦只能写在**根 link** 上（该 link 的**全部** collision 都会拿到这个 μ）。
+             物理上没关系：真正接地的只有 4 个轮 cylinder（整车最低点 −0.1025 m 在轮上），
+             其余 box 的最低点都在 −0.0780 m 以上、正常姿态下永不触地。
+       代价（**故意改的物理，不是几何**）：轮子对地静摩擦角 = atan(0.02) ≈ **1.1°** ⇒ 在更陡的坡上
+       停住会缓慢下滑（平面速度驱动爬坡不受影响，插件直接设速度、不需要抓地）。要更抓地就重新生成：
+       `—wheel-mu 0.1`（→ 自转 ≈82.3%、≈5.7° 坡）或 `—wheel-mu 0.05`（→ ≈89.6%、≈2.9°）。
+       生成：`python3 tools/scripts/regress/robot11_make_sim_xacro.py —wheel-mu 0.02`（缺省即此值）；
+       `—wheel-mu 0` 或 `—no-wheel-friction` = 回到"缺省 μ=1"的改前行为（不写这一块）。 -->
+  <gazebo reference="base_link">
+    <mu1>0.02</mu1>
+    <mu2>0.02</mu2>
+  </gazebo>
   <!-- ==================== 几何速查（实测值，来自 Phase 1/3；供 config 对照） ====================
        地面平面（body 系） z = **-0.102499**（四个轮 mesh 的最低点；轮 r=0.0580 心在 z=-0.0445）
@@ -872,3 +896,9 @@
        回退：`robot11_make_sim_xacro.py —chassis articulated` —— 模型体（去注释）
        逐字节相同（实测 35025 B vs 35025 B），文件只多出文件头那段说明。
+       ★ 2026-10-20：**轮子对地摩擦 μ=0.02**（`<gazebo reference="base_link">` 的 mu1/mu2；
+       写在 `<link>` 里的 mu1/mu2 Gazebo **不认**）。上面那个 16.5% 是"只塌刚体、
+       不加摩擦"的旧数字；加摩擦后同一台架纯自转 wz=0.8 → **95.8%**
+       （改前 10.6%；整栈 20 Hz 9.8% → **92.9%**、200 Hz 95.3%）。几何一个字节没动，由
+       `gz sdf -p` 的逐条 AABB + 质量/Izz 自证。代价：静摩擦角 ≈ 1.1°，更陡的坡上
+       停住会滑（速度驱动爬坡不受影响）。剂量-响应/下游冒烟见 docs §22。
 --></robot>

Commit message: feat(frames): 按实车改雷达安装约定 —— base_link→livox_frame rpy=0、倾角搬到 livox_frame→imu_link、LIO extrinsic_R 从 URDF 注入（契约 §4.12）
实车：Livox 驱动的 extrinsic_parameter 只旋点云（IMU 通路另一套单位阵 extrinsic_global），TF base_link→livox_frame rpy=0。
sim 复现：关节 rpy=0（只有平移，几何逐位不变）；倾角放 livox_frame→imu_link（IMU 真的斜 30°，offset 也跟着转 ⇒ base_link→imu_link 与改动前逐位相同）；插件 <tilt_rpy> 旋射线并把点旋进水平的 livox_frame（插件代码一行没改，出点公式本来就表达在 frame_id 帧里）；LIO 外参由 launch 从 URDF 解析注入（extrinsic_R=Rx(+30°)、extrinsic_T=[0,0,0.05] 不变）；gravity_align_rpy 改从 IMU 链取（值不变）。
附带修 small_point_lio 的 off 分支 latent bug：初始地图原先把雷达系点原样入图（= 假设 R_IL=I），新约定会发散（实测 map→odom 1e5 m / score=nan）；R_IL=I 时仍走原表达式（逐字节不变）。
robot11_mount 收敛成唯一值 sensor（plugin/urdf 两个实验臂删除，传了硬报错）。

File: src/rm_nav_bringup/urdf/sentry_robot_robot11_sim.xacro (robot description, xacro)
@@ -48,15 +48,27 @@
        `<cloud_frame>` 元素；它的两处 property 取值与 urdf 档完全相同）—— 见 §J 的静态证据。
        ========================================================================== -->
-  <xacro:arg name="livox_mount" default="plugin" />
-  <xacro:property name="livox_mount_p" value="$(arg livox_mount)" />
+  <xacro:arg name="livox_mount" default="sensor" />
   <xacro:property name="livox_tilt_rpy_p" value="$(arg livox_tilt_rpy)" />
-  <!-- 倾角记在**关节**上的两档（urdf / sensor）：关节 rpy = 倾角、插件 <tilt_rpy> = 单位阵 -->
-  <xacro:property name="livox_mount_tilt_in_joint" value="${livox_mount_p.strip() in ('urdf', 'sensor')}" />
-  <!-- 点云表达在**传感器系**的那一档（sensor；缺省/plugin/urdf = 父 link 系） -->
-  <xacro:property name="livox_mount_sensor" value="${livox_mount_p.strip() == 'sensor'}" />
-  <!-- 关节 rpy：urdf/sensor 档 = 倾角；plugin 档 = 0 -->
-  <xacro:property name="livox_joint_rpy" value="${livox_tilt_rpy_p if livox_mount_tilt_in_joint else '0 0 0'}" />
-  <!-- 插件 <tilt_rpy>：plugin 档 = 倾角；urdf/sensor 档 = 单位阵（射线已由 link 姿态带斜） -->
-  <xacro:property name="livox_plugin_tilt_rpy" value="${'0 0 0' if livox_mount_tilt_in_joint else livox_tilt_rpy_p}" />
+  <!-- ★★★ 2026-10-21（**按实车改约定**）：`livox_mount` 已**不再改变几何**（只剩一个值 `sensor`，
+       见文件头的"实车约定"）。下面四条 property 因此是**常量**，保留成 property 只是为了让
+       下游（`<joint>` / `<sensor>`）的引用不动。 -->
+  <xacro:property name="livox_mount_tilt_in_joint" value="False" />
+  <xacro:property name="livox_mount_sensor" value="False" />
+  <!-- 关节 rpy：**永远 0**（`base_link→livox_frame` 只有平移 ⇒ 与实车的 TF 一致） -->
+  <xacro:property name="livox_joint_rpy" value="0 0 0" />
+  <!-- 插件 <tilt_rpy>：**永远 = 倾角**（射线真的斜；点按"实车驱动器的做法"旋进这个水平帧，
+       见 livox_points_plugin.cpp 的出点公式：`point = (range+minDist)·(mount_rot·ray·x̂)`）。 -->
+  <xacro:property name="livox_plugin_tilt_rpy" value="${livox_tilt_rpy_p}" />
+  <!-- IMU 的安装偏移（在 `livox_frame` 里）：`Rx(r)·Ry(p)·Rz(y) · (0,0,-0.05)`。
+       为什么要在 xacro 里算：`imu_joint` 现在是**唯一**知道"IMU 相对雷达斜 30°"的地方
+       （TF：`base_link→livox_frame` rpy=0、`livox_frame→imu_link` rpy=倾角），
+       而 IMU 的**物理位置**必须与改动前逐位相同 ⇒ 偏移要跟着倾角转。 -->
+  <xacro:property name="livox_tilt_vals" value="${[float(v) for v in livox_tilt_rpy_p.split()]}" />
+  <xacro:property name="tr" value="${livox_tilt_vals[0]}" />
+  <xacro:property name="tp" value="${livox_tilt_vals[1]}" />
+  <xacro:property name="ty" value="${livox_tilt_vals[2]}" />
+  <xacro:property name="imu_v1" value="${(0.0, 0.05 * sin(tr), -0.05 * cos(tr))}" />
+  <xacro:property name="imu_v2" value="${(imu_v1[0] * cos(tp) + imu_v1[2] * sin(tp), imu_v1[1],                            -imu_v1[0] * sin(tp) + imu_v1[2] * cos(tp))}" />
+  <xacro:property name="imu_v3" value="${(imu_v2[0] * cos(ty) - imu_v2[1] * sin(ty),                            imu_v2[0] * sin(ty) + imu_v2[1] * cos(ty), imu_v2[2])}" />
   <!-- ==========================================================================
        【我们加的｜Phase 5（2026-10-07）】`<visual>` 用哪一档 mesh —— **只改渲染代价，不改几何**
@@ -707,7 +719,14 @@
          (c) 后果（IMU 的 z 轴相对 base_link 斜 30°）由 `lio_tf_adapter` 的 `rpy` 精确补偿，
              已在本槽位的 launch 分支里显式写死并实测（见 docs/robot_models.md §10）。
-       绝对位置：body + (0.000562, 0.130916, 0.107028)（= 雷达原点沿**雷达自身的** −z 走 0.05 m）。 -->
+       ★★ 2026-10-21（**按实车改约定**）：`base_link→livox_frame` 现在 rpy=0（只有平移），
+       倾角搬到**这一条**（`livox_frame→imu_link`）⇒ IMU 物理上仍然斜 30°（加速度计真的感受到），
+       而点云在**水平**的 `livox_frame` 里（与实车驱动器把点云旋进机器人系的语义一致）。
+       为了"物理几何一个字节都不变"，偏移也要跟着倾角转：
+         xyz = Rx(r)·Ry(p)·Rz(y)·(0,0,-0.05)   （r,p,y = `livox_tilt_rpy`）
+       于是 `base_link→imu_link` 与改动前**逐位相同**（rpy = 倾角、位置 = 雷达原点沿雷达到 IMU
+       的 −z 走 0.05 m）；`h_imu` 不变、静态边 `odom→odom_level` 的值也不变。
+       三条一致性（driver/插件 = TF 的旋转 + LIO 外参）见 docs/frame_contract_v3.md §4.12。 -->
   <joint name="imu_joint" type="fixed">
-    <origin xyz="0 0 -0.05" rpy="0 0 0" />
+    <origin xyz="${imu_v3[0]} ${imu_v3[1]} ${imu_v3[2]}" rpy="${livox_tilt_rpy_p}" />
     <parent link="livox_frame" />
     <child link="imu_link" />

Commit message: feat(livox): 雷达按实车拆成"物理斜装 + 驱动器外参"两层（livox_physical + livox_cloud_extrinsic）
用户原话："模型斜，点云也倾斜，然后改之前说的那个外参给点云转正"。

模型（generator + 生成的 xacro 同步改）：
- 新增 link `livox_physical`（`l12` 的 visual + 上游惯量、**无 collision**）+ 关节
  `body_to_livox_physical`（parent=base_link、xyz 与 body_to_livox 逐字相同、rpy = livox_tilt_rpy = -30°）
  ⇒ **画出来的雷达真的斜**；射线传感器挂这里。
- `livox_frame` 变成**纯数据帧**（rpy=0、无几何、1e-6 占位惯量）。
- 插件：`<gazebo reference="livox_physical">`、`<sensor name="livox_physical">`、`<tilt_rpy>0 0 0</tilt_rpy>`
  （倾角由 link 姿态承担）⇒ 原始点云表达在**斜的物理系**，话题 `/livox/lidar_raw`。
- `livox_frame→imu_link` 仍是 rpy=-30°（IMU 物理上斜）⇒ h_imu / §4.11 静态边 / LIO extrinsic_R 全不变。

驱动器外参（新节点 `livox_cloud_extrinsic`，cloud_accumulator 包）：
- 旋转**从 TF 读** `livox_frame←livox_physical`（= Rx(+30°)，唯一真源 = URDF），TF 拿不到才退参数；
- 输出**两种消息**：`/livox/lidar`（CustomMsg，LIO 吃）**和** `/livox/lidar/pointcloud`（PointCloud2，
  linefit/accumulator/p2l 吃），`frame_id=livox_frame`；CustomMsg 走**就地逐点旋转**（不新建 3 万对象）。
- launch：`bringup_sim.launch.py` 在 linefit 之前加这个节点；横幅文案同步。

⚠️ 第一次接线把数据链接断了（已修，measurements §47.1 复盘）：
  /livox/lidar_raw 是 CustomMsg（**BEST_EFFORT**）、/livox/lidar_raw/pointcloud 才是 PointCloud2；
  第一版用 PointCloud2 订阅 raw、且只发 /livox/lidar 一种类型 ⇒ LIO 与 linefit/accumulator **同时断流**；
  第二版 CustomMsg 订阅用 RELIABLE 与插件的 BEST_EFFORT **不兼容** ⇒ /livox/lidar 仍 0 Hz。

实测（headless，robot:=robot11 world:=RMUC2026，ROS_DOMAIN_ID 隔离）：
- `/livox/lidar_raw` CustomMsg 4.28 Hz（pub=livox_physical_plugin BEST_EFFORT、sub=livox_cloud_extrinsic）
- `/livox/lidar` CustomMsg **4.49 Hz**（pub=livox_cloud_extrinsic RELIABLE）
- `/livox/lidar/pointcloud` PointCloud2 **4.44 Hz**；`/livox/imu` 36.1 Hz（本机 RTF≈0.43，比率自洽）
- TF `base_link→livox_frame` RPY (0,0,0)、`base_link→livox_physical` RPY (-0.524,0,0)
- 地面法向：原始云 `[+0.0006,-0.5023,+0.8647]` = **30.15°**；转正后 `[+0.0006,-0.0020,+1.0000]` = **0.12°**
- `/robot_description`：robot_state_publisher 以 TRANSIENT_LOCAL+RELIABLE 发布（与 nav2.rviz 的
  RobotModel 配置一致；install 里是指向源码的符号链接）

docs：契约新增 §4.12.6（两层分解 + 消息类型/QoS 契约），§4.12.2 两行同步；measurements 新增 §47
（分解/断线复盘/实测/诚实清单）；robot_models §9.0（mesh 归属变了：l12 现在画在 livox_physical 上）。

File: src/rm_nav_bringup/urdf/sentry_robot_robot11_sim.xacro (robot description, xacro)
@@ -638,5 +638,19 @@
   <!-- ==================== link livox_frame ==================== -->
   <link name="livox_frame">
-    <!-- 【上游原样】inertial -->
+    <!-- ★ 2026-10-29：本 link 现在是**纯数据帧**（`base_link→livox_frame` rpy=0，与实车 TF 一致）。
+         几何（mesh/inertial）搬到 `livox_physical`；点云由 `livox_cloud_extrinsic` 从
+         `/livox/lidar_raw`（斜的物理系）旋 `Rx(+倾角)` 到本帧后发 `/livox/lidar`。
+         为什么留一个极小惯量：Gazebo 对"固定关节链上的无惯量 link"会走 lumping 告警路径，
+         给个 1e-6 量级的占位最省事（物理质量在 livox_physical 上，总质量不变）。 -->
+    <inertial>
+      <origin xyz="0 0 0" rpy="0 0 0" />
+      <mass value="1e-6" />
+      <inertia ixx="1e-9" ixy="0" ixz="0" iyy="1e-9" iyz="0" izz="1e-9" />
+    </inertial>
+  </link>
+  <!-- ==================== link livox_physical（2026-10-29 新增：物理雷达） ==================== -->
+  <link name="livox_physical">
+    <!-- 物理本体：inertial + mesh 都从 livox_frame 搬过来（逐字），**故意不给 collision**
+         （射线传感器就在本 link 原点，给碰撞体 ⇒ 每条射线打自己；docs/robot_models.md §10.5）。 -->
     <inertial>
       <origin xyz="-0.000348524070196802 0.00208606529928732 0.0221378690951775" rpy="0 0 0" />
@@ -644,5 +658,4 @@
       <inertia ixx="4.17032187760686E-05" ixy="-5.98077892665089E-09" ixz="3.05517185056836E-07" iyy="4.50191700802289E-05" iyz="-5.90930308926011E-10" izz="6.87178468496533E-05" />
     </inertial>
-    <!-- 【上游原样】visual（几何位置/单位/材质逐字照抄；mesh 文件按 `visual_dir` 换档，见文件头 Phase 5） -->
     <visual>
       <origin xyz="0 0 0" rpy="0 0 0" />
@@ -650,6 +663,4 @@
       <material name=""><color rgba="0.792156862745098 0.819607843137255 0.933333333333333 1" /></material>
     </visual>
-    <!-- 【我们加的｜替换】上游这里是 mesh collision；按 Phase 1 实测换掉（原因见文件头） -->
-    <!-- livox_frame：**故意不给 collision**（射线传感器就在本 link 原点上，给碰撞体 = 每条射线打自己；实测见 docs/robot_models.md §10.5） -->
   </link>
   <!-- ==================== joint j2 ==================== -->
@@ -706,4 +717,14 @@
     <axis xyz="0 0 0" />
   </joint>
+  <!-- ==================== joint body_to_livox_physical（2026-10-29 新增） ==================== -->
+  <!-- 物理安装姿态：`base_link→livox_physical` 的 rpy = `livox_tilt_rpy`（实车的 −30° 下俯），
+       xyz 与 `body_to_livox` **逐字相同**（雷达的物理位置没动，只是把 30° 从插件参数搬到 link 上）。
+       ⇒ 射线方向不变（世界系里逐条相同），但**点云表达在斜系**（`/livox/lidar_raw`），
+       与实车驱动器"原始点云在传感器系"一致。 -->
+  <joint name="body_to_livox_physical" type="fixed">
+    <origin xyz="0.000561701465058485 0.130915824456595 ${0.15702816968305 + livox_raise_m_p}" rpy="${livox_tilt_rpy_p}" />
+    <parent link="base_link" />
+    <child link="livox_physical" />
+  </joint>
   <!-- ==================== 【我们加的】配件：IMU / 雷达 / 底盘 ==================== -->
   <!-- 上游 URDF 里**没有** imu_link、没有 <gazebo>、没有 <sensor>、没有 <plugin>
@@ -756,11 +777,11 @@
        射线参数与宏一致：水平 100 × 垂直 360、10 Hz、0.1–200 m、σ=2 mm、
        垂直 FOV −7.22°…+55.22°（这是本仓 mid360.xacro 的既有取值）。 -->
-  <gazebo reference="livox_frame">
-    <sensor type="ray" name="livox_frame">
+  <gazebo reference="livox_physical">
+    <sensor type="ray" name="livox_physical">
       <pose>0 0 0 0 0 0</pose>
       <always_on>true</always_on>
       <visualize>false</visualize>
       <update_rate>10</update_rate>
-      <plugin name="livox_frame_plugin" filename="libros2_livox.so">
+      <plugin name="livox_physical_plugin" filename="libros2_livox.so">
         <ray>
           <scan>
@@ -799,9 +820,10 @@
              $(arg livox_tilt_rpy)（下面这条，与 2026-10-07 逐字节相同）；
              urdf/sensor 档 = `0 0 0`（倾角已经写在关节上，射线由 link 姿态带斜）。 -->
-        <tilt_rpy>${livox_plugin_tilt_rpy}</tilt_rpy>
+        <!-- 0 0 0：倾角改由 `body_to_livox_physical` 的关节 rpy 承担（2026-10-29） -->
+        <tilt_rpy>0 0 0</tilt_rpy>
         <samples>30000</samples>
         <downsample>1</downsample>
         <csv_file_name>$(find ros2_livox_simulation)/scan_mode/mid360.csv</csv_file_name>
-        <topic>/livox/lidar</topic><!--【我们加的｜2026-10-09】`livox_mount:=sensor` 档才发下面这个元素（**写在行内**：
+        <topic>/livox/lidar_raw</topic><!--【我们加的｜2026-10-09】`livox_mount:=sensor` 档才发下面这个元素（**写在行内**：
              条件为假时 xacro 连同它的缩进一起删掉 ⇒ plugin/urdf 两档的渲染去注释后逐字节不变）。
              语义（`livox_points_plugin.cpp` 的 `cloud_frame_sensor_`）：点云表达在**真·传感器系**
@@ -853,5 +875,5 @@
   <!-- ⑤ 材质（纯观感） -->
   <gazebo reference="base_link"><material>Gazebo/Orange</material></gazebo>
-  <gazebo reference="livox_frame"><material>Gazebo/LightBlueLaser</material></gazebo>
+  <gazebo reference="livox_physical"><material>Gazebo/LightBlueLaser</material></gazebo>
   <gazebo reference="imu_link"><material>Gazebo/BuildingFrame</material></gazebo>
   <!-- ⑥ 【我们加的｜2026-10-20】**轮子对地摩擦**（★ Gazebo 只认 `<gazebo reference>` 这一种写法）
@@ -907,5 +929,5 @@
        把 11 个 link（base_link, l10, l11, l2, l3, l4, l5, l6, l7, l8, l9）塌成 1 个刚体：碰撞/视觉几何**逐条**搬进根 link，
        质量/质心/惯量按平行轴定理合成（M=9.4121 kg、Izz=0.12677 kg·m²）；
-       删掉 10 个关节（j2…j11），**保留** livox_frame/imu_link 与它们的固定关节。
+       删掉 10 个关节（j2…j11），**保留** livox_frame/livox_physical/imu_link 与它们的固定关节。
        为什么（实测，见 docs/tilted_lidar_fidelity.md §M）：planar_move 是
        `Model::Set*Vel` = 把同一个 (v,ω) 写给**每一个 link**，只有单刚体才自洽；
