Commit message: fix(robot): 起伏底盘轮子改 continuous 被动滚动（同默认模型），去固定轮 μ=0.02 特殊处理

File: src/rm_nav_bringup/urdf/sentry_robot_chassis_boxvis_sim.xacro (robot description, xacro)
@@ -53,9 +53,11 @@
       </collision>
     </link>
-    <joint name="${name}" type="fixed">
+    <joint name="${name}" type="continuous">
       <origin xyz="${xyz}" rpy="0 0 0" />
       <parent link="base_link" />
       <child link="${name}" />
-      <axis xyz="0 0 0" />
+      <!-- 轮轴 = 轮子坐标系 y（轮 mesh 的轴向；collision 圆柱 rpy=+90° 也把轴转到 y）
+           ⇒ 轮子**被动滚动**（与默认模型一致，无轮控制器；底盘由 planar_move 驱动）。 -->
+      <axis xyz="0 1 0" />
     </joint>
   </xacro:macro>
@@ -83,8 +85,8 @@
     </plugin>
   </gazebo>
-  <gazebo reference="w1"><mu1>0.02</mu1><mu2>0.02</mu2></gazebo>
-  <gazebo reference="w2"><mu1>0.02</mu1><mu2>0.02</mu2></gazebo>
-  <gazebo reference="w3"><mu1>0.02</mu1><mu2>0.02</mu2></gazebo>
-  <gazebo reference="w4"><mu1>0.02</mu1><mu2>0.02</mu2></gazebo>
+  <gazebo reference="w1"><mu1>0.8</mu1><mu2>0.8</mu2></gazebo>
+  <gazebo reference="w2"><mu1>0.8</mu1><mu2>0.8</mu2></gazebo>
+  <gazebo reference="w3"><mu1>0.8</mu1><mu2>0.8</mu2></gazebo>
+  <gazebo reference="w4"><mu1>0.8</mu1><mu2>0.8</mu2></gazebo>
   <!-- ===================== IMU（平放） ===================== -->
   <link name="imu_link" />

File: src/rm_nav_bringup/urdf/sentry_robot_chassis_sim.xacro (robot description, xacro)
@@ -53,9 +53,11 @@
       </collision>
     </link>
-    <joint name="${name}" type="fixed">
+    <joint name="${name}" type="continuous">
       <origin xyz="${xyz}" rpy="0 0 0" />
       <parent link="base_link" />
       <child link="${name}" />
-      <axis xyz="0 0 0" />
+      <!-- 轮轴 = 轮子坐标系 y（轮 mesh 的轴向；collision 圆柱 rpy=+90° 也把轴转到 y）
+           ⇒ 轮子**被动滚动**（与默认模型一致，无轮控制器；底盘由 planar_move 驱动）。 -->
+      <axis xyz="0 1 0" />
     </joint>
   </xacro:macro>
@@ -83,12 +85,10 @@
     </plugin>
   </gazebo>
-  <!-- 轮子对地摩擦：planar_move 直接设速度、轮子**不转**（固定关节）⇒ 若轮子高摩擦
-       （默认 μ=1）会在加速/转向时"抓住"地面把车**掀翻**（实测：起步/急转就翻）。
-       与 robot11 同款处理：4 个轮子的 collision 都降到 μ=0.02（轮子滑动而不是抓地），
-       底盘由 planar_move 直接驱动 ⇒ 不再翻车。base_link 的 box 离地 0.08 m，不触地。 -->
-  <gazebo reference="w1"><mu1>0.02</mu1><mu2>0.02</mu2></gazebo>
-  <gazebo reference="w2"><mu1>0.02</mu1><mu2>0.02</mu2></gazebo>
-  <gazebo reference="w3"><mu1>0.02</mu1><mu2>0.02</mu2></gazebo>
-  <gazebo reference="w4"><mu1>0.02</mu1><mu2>0.02</mu2></gazebo>
+  <!-- 轮子：**continuous 被动滚动**（与默认模型同款，无轮控制器）⇒ 不需要把摩擦降到 0.02
+       （那是"焊接固定轮"才需要的）；滚动轮随地面滚动，planar_move 驱动底盘，不会因"抓地"掀翻。 -->
+  <gazebo reference="w1"><mu1>0.8</mu1><mu2>0.8</mu2></gazebo>
+  <gazebo reference="w2"><mu1>0.8</mu1><mu2>0.8</mu2></gazebo>
+  <gazebo reference="w3"><mu1>0.8</mu1><mu2>0.8</mu2></gazebo>
+  <gazebo reference="w4"><mu1>0.8</mu1><mu2>0.8</mu2></gazebo>
   <!-- ===================== IMU（平放） ===================== -->
   <link name="imu_link" />

Commit message: revert(robot): 起伏底盘轮子回固定轮+μ0.02（连续被动轮上不了坡）；视觉回原始 STL（排查轮子不显示）

File: src/rm_nav_bringup/urdf/sentry_robot_chassis_boxvis_sim.xacro (robot description, xacro)
@@ -53,11 +53,9 @@
       </collision>
     </link>
-    <joint name="${name}" type="continuous">
+    <joint name="${name}" type="fixed">
       <origin xyz="${xyz}" rpy="0 0 0" />
       <parent link="base_link" />
       <child link="${name}" />
-      <!-- 轮轴 = 轮子坐标系 y（轮 mesh 的轴向；collision 圆柱 rpy=+90° 也把轴转到 y）
-           ⇒ 轮子**被动滚动**（与默认模型一致，无轮控制器；底盘由 planar_move 驱动）。 -->
-      <axis xyz="0 1 0" />
+      <axis xyz="0 0 0" />
     </joint>
   </xacro:macro>

File: src/rm_nav_bringup/urdf/sentry_robot_chassis_sim.xacro (robot description, xacro)
@@ -23,5 +23,5 @@
     <visual>
       <origin xyz="0 0 0" rpy="0 0 0" />
-      <geometry><mesh filename="package://chassis_description/meshes/decimated/base_link.stl" /></geometry>
+      <geometry><mesh filename="package://chassis_description/meshes/base_link.STL" /></geometry>
       <material name="chassis_body"><color rgba="0.792 0.820 0.933 1" /></material>
     </visual>
@@ -45,5 +45,5 @@
       <visual>
         <origin xyz="0 0 0" rpy="0 0 0" />
-        <geometry><mesh filename="package://chassis_description/meshes/decimated/${name}.stl" /></geometry>
+        <geometry><mesh filename="package://chassis_description/meshes/${name}.STL" /></geometry>
         <material name="wheel_white"><color rgba="1 1 1 1" /></material>
       </visual>
@@ -53,11 +53,9 @@
       </collision>
     </link>
-    <joint name="${name}" type="continuous">
+    <joint name="${name}" type="fixed">
       <origin xyz="${xyz}" rpy="0 0 0" />
       <parent link="base_link" />
       <child link="${name}" />
-      <!-- 轮轴 = 轮子坐标系 y（轮 mesh 的轴向；collision 圆柱 rpy=+90° 也把轴转到 y）
-           ⇒ 轮子**被动滚动**（与默认模型一致，无轮控制器；底盘由 planar_move 驱动）。 -->
-      <axis xyz="0 1 0" />
+      <axis xyz="0 0 0" />
     </joint>
   </xacro:macro>
@@ -85,10 +83,11 @@
     </plugin>
   </gazebo>
-  <!-- 轮子：**continuous 被动滚动**（与默认模型同款，无轮控制器）⇒ 不需要把摩擦降到 0.02
-       （那是"焊接固定轮"才需要的）；滚动轮随地面滚动，planar_move 驱动底盘，不会因"抓地"掀翻。 -->
-  <gazebo reference="w1"><mu1>0.8</mu1><mu2>0.8</mu2></gazebo>
-  <gazebo reference="w2"><mu1>0.8</mu1><mu2>0.8</mu2></gazebo>
-  <gazebo reference="w3"><mu1>0.8</mu1><mu2>0.8</mu2></gazebo>
-  <gazebo reference="w4"><mu1>0.8</mu1><mu2>0.8</mu2></gazebo>
+  <!-- 轮子：**固定轮**（与 robot11 同款处理）——4 轮用 μ=0.02 **滑动**而不是抓地，
+       底盘由 planar_move 直接驱动（速度驱动，爬坡靠"直接设速度"、不靠抓地）；
+       高摩擦固定轮会被加速/转向掀翻（实测）。 -->
+  <gazebo reference="w1"><mu1>0.02</mu1><mu2>0.02</mu2></gazebo>
+  <gazebo reference="w2"><mu1>0.02</mu1><mu2>0.02</mu2></gazebo>
+  <gazebo reference="w3"><mu1>0.02</mu1><mu2>0.02</mu2></gazebo>
+  <gazebo reference="w4"><mu1>0.02</mu1><mu2>0.02</mu2></gazebo>
   <!-- ===================== IMU（平放） ===================== -->
   <link name="imu_link" />

Commit message: feat(robot): 起伏底盘改真轮驱动（diff_drive：w1/w2 驱动、w3/w4 被动；扭矩 5 N·m）

File: src/rm_nav_bringup/urdf/sentry_robot_chassis_boxvis_sim.xacro (robot description, xacro)
@@ -53,9 +53,10 @@
       </collision>
     </link>
-    <joint name="${name}" type="fixed">
+    <joint name="${name}" type="continuous">
       <origin xyz="${xyz}" rpy="0 0 0" />
       <parent link="base_link" />
       <child link="${name}" />
-      <axis xyz="0 0 0" />
+      <!-- 轮轴 = 轮子坐标系 y（轮 mesh 的轴向；collision 圆柱 rpy=+90° 也把轴转到 y） -->
+      <axis xyz="0 1 0" />
     </joint>
   </xacro:macro>
@@ -65,6 +66,9 @@
   <xacro:chassis_wheel name="w4" xyz="-0.1615 0.10895 -0.04" />
   <!-- ===================== 驱动 + 真值里程计（与 robot11 同款） ===================== -->
+  <!-- ★ 2026-10-30：真轮驱动（diff_drive）——planar_move 换成"轮子扭矩"：
+       前轮 w1(左)/w2(右) 由差速插件驱动，后轮 w3/w4 连续被动滚动。
+       轮径 0.116 m、轮距 0.281 m；扭矩上限 5 N·m、加速度上限 2 m/s²（防起步掀翻）。 -->
   <gazebo>
-    <plugin name="mecanum_controller" filename="libgazebo_ros_planar_move.so">
+    <plugin name="diff_drive" filename="libgazebo_ros_diff_drive.so">
       <ros>
         <namespace>/</namespace>
@@ -73,12 +77,17 @@
       </ros>
       <update_rate>100</update_rate>
-      <publish_rate>10</publish_rate>
+      <left_joint>w1</left_joint>
+      <right_joint>w2</right_joint>
+      <wheel_separation>0.281</wheel_separation>
+      <wheel_diameter>0.116</wheel_diameter>
+      <max_wheel_torque>5.0</max_wheel_torque>
+      <max_wheel_acceleration>2.0</max_wheel_acceleration>
+      <command_topic>cmd_vel</command_topic>
+      <odometry_topic>odom</odometry_topic>
+      <odometry_frame>odom</odometry_frame>
+      <robot_base_frame>base_link</robot_base_frame>
       <publish_odom>true</publish_odom>
       <publish_odom_tf>false</publish_odom_tf>
-      <odometry_frame>odom</odometry_frame>
-      <robot_base_frame>base_link</robot_base_frame>
-      <covariance_x>0.0001</covariance_x>
-      <covariance_y>0.0001</covariance_y>
-      <covariance_yaw>0.01</covariance_yaw>
+      <publish_wheel_tf>true</publish_wheel_tf>
     </plugin>
   </gazebo>

File: src/rm_nav_bringup/urdf/sentry_robot_chassis_sim.xacro (robot description, xacro)
@@ -53,9 +53,10 @@
       </collision>
     </link>
-    <joint name="${name}" type="fixed">
+    <joint name="${name}" type="continuous">
       <origin xyz="${xyz}" rpy="0 0 0" />
       <parent link="base_link" />
       <child link="${name}" />
-      <axis xyz="0 0 0" />
+      <!-- 轮轴 = 轮子坐标系 y（轮 mesh 的轴向；collision 圆柱 rpy=+90° 也把轴转到 y） -->
+      <axis xyz="0 1 0" />
     </joint>
   </xacro:macro>
@@ -65,6 +66,9 @@
   <xacro:chassis_wheel name="w4" xyz="-0.1615 0.10895 -0.04" />
   <!-- ===================== 驱动 + 真值里程计（与 robot11 同款） ===================== -->
+  <!-- ★ 2026-10-30：真轮驱动（diff_drive）——planar_move 换成"轮子扭矩"：
+       前轮 w1(左)/w2(右) 由差速插件驱动，后轮 w3/w4 连续被动滚动。
+       轮径 0.116 m、轮距 0.281 m；扭矩上限 5 N·m、加速度上限 2 m/s²（防起步掀翻）。 -->
   <gazebo>
-    <plugin name="mecanum_controller" filename="libgazebo_ros_planar_move.so">
+    <plugin name="diff_drive" filename="libgazebo_ros_diff_drive.so">
       <ros>
         <namespace>/</namespace>
@@ -73,12 +77,17 @@
       </ros>
       <update_rate>100</update_rate>
-      <publish_rate>10</publish_rate>
+      <left_joint>w1</left_joint>
+      <right_joint>w2</right_joint>
+      <wheel_separation>0.281</wheel_separation>
+      <wheel_diameter>0.116</wheel_diameter>
+      <max_wheel_torque>5.0</max_wheel_torque>
+      <max_wheel_acceleration>2.0</max_wheel_acceleration>
+      <command_topic>cmd_vel</command_topic>
+      <odometry_topic>odom</odometry_topic>
+      <odometry_frame>odom</odometry_frame>
+      <robot_base_frame>base_link</robot_base_frame>
       <publish_odom>true</publish_odom>
       <publish_odom_tf>false</publish_odom_tf>
-      <odometry_frame>odom</odometry_frame>
-      <robot_base_frame>base_link</robot_base_frame>
-      <covariance_x>0.0001</covariance_x>
-      <covariance_y>0.0001</covariance_y>
-      <covariance_yaw>0.01</covariance_yaw>
+      <publish_wheel_tf>true</publish_wheel_tf>
     </plugin>
   </gazebo>
@@ -86,8 +95,8 @@
        底盘由 planar_move 直接驱动（速度驱动，爬坡靠"直接设速度"、不靠抓地）；
        高摩擦固定轮会被加速/转向掀翻（实测）。 -->
-  <gazebo reference="w1"><mu1>0.02</mu1><mu2>0.02</mu2></gazebo>
-  <gazebo reference="w2"><mu1>0.02</mu1><mu2>0.02</mu2></gazebo>
-  <gazebo reference="w3"><mu1>0.02</mu1><mu2>0.02</mu2></gazebo>
-  <gazebo reference="w4"><mu1>0.02</mu1><mu2>0.02</mu2></gazebo>
+  <gazebo reference="w1"><mu1>0.8</mu1><mu2>0.8</mu2></gazebo>
+  <gazebo reference="w2"><mu1>0.8</mu1><mu2>0.8</mu2></gazebo>
+  <gazebo reference="w3"><mu1>0.8</mu1><mu2>0.8</mu2></gazebo>
+  <gazebo reference="w4"><mu1>0.8</mu1><mu2>0.8</mu2></gazebo>
   <!-- ===================== IMU（平放） ===================== -->
   <link name="imu_link" />
