Commit message: perf(robot): 起伏底盘视觉减面（base 20k->8k、轮 8k->2.5k，平滑 LOD）+ 碰撞改基本体（box+cylinder，隐藏）

File: src/rm_nav_bringup/urdf/sentry_robot_chassis_sim.xacro (robot description, xacro)
@@ -26,5 +26,5 @@
       <geometry>
         <mesh
-          filename="package://chassis_description/meshes/base_link.STL" />
+          filename="package://chassis_description/meshes/decimated/base_link.stl" />
       </geometry>
       <material
@@ -35,11 +35,6 @@
     </visual>
     <collision>
-      <origin
-        xyz="0 0 0"
-        rpy="0 0 0" />
-      <geometry>
-        <mesh
-          filename="package://chassis_description/meshes/base_link.STL" />
-      </geometry>
+      <origin xyz="0 0 0.0295" rpy="0 0 0" />
+      <geometry><box size="0.456 0.446 0.097" /></geometry>
     </collision>
   </link>
@@ -66,20 +61,15 @@
       <geometry>
         <mesh
-          filename="package://chassis_description/meshes/w1.STL" />
-      </geometry>
-      <material
-        name="">
-        <color
-          rgba="1 1 1 1" />
-      </material>
-    </visual>
-    <collision>
-      <origin
-        xyz="0 0 0"
-        rpy="0 0 0" />
-      <geometry>
-        <mesh
-          filename="package://chassis_description/meshes/w1.STL" />
-      </geometry>
+          filename="package://chassis_description/meshes/decimated/w1.stl" />
+      </geometry>
+      <material
+        name="">
+        <color
+          rgba="1 1 1 1" />
+      </material>
+    </visual>
+    <collision>
+      <origin xyz="0 -0.032 0" rpy="1.5707963 0 0" />
+      <geometry><cylinder radius="0.058" length="0.03" /></geometry>
     </collision>
   </link>
@@ -119,20 +109,15 @@
       <geometry>
         <mesh
-          filename="package://chassis_description/meshes/w2.STL" />
-      </geometry>
-      <material
-        name="">
-        <color
-          rgba="1 1 1 1" />
-      </material>
-    </visual>
-    <collision>
-      <origin
-        xyz="0 0 0"
-        rpy="0 0 0" />
-      <geometry>
-        <mesh
-          filename="package://chassis_description/meshes/w2.STL" />
-      </geometry>
+          filename="package://chassis_description/meshes/decimated/w2.stl" />
+      </geometry>
+      <material
+        name="">
+        <color
+          rgba="1 1 1 1" />
+      </material>
+    </visual>
+    <collision>
+      <origin xyz="0 -0.032 0" rpy="1.5707963 0 0" />
+      <geometry><cylinder radius="0.058" length="0.03" /></geometry>
     </collision>
   </link>
@@ -172,20 +157,15 @@
       <geometry>
         <mesh
-          filename="package://chassis_description/meshes/w3.STL" />
-      </geometry>
-      <material
-        name="">
-        <color
-          rgba="1 1 1 1" />
-      </material>
-    </visual>
-    <collision>
-      <origin
-        xyz="0 0 0"
-        rpy="0 0 0" />
-      <geometry>
-        <mesh
-          filename="package://chassis_description/meshes/w3.STL" />
-      </geometry>
+          filename="package://chassis_description/meshes/decimated/w3.stl" />
+      </geometry>
+      <material
+        name="">
+        <color
+          rgba="1 1 1 1" />
+      </material>
+    </visual>
+    <collision>
+      <origin xyz="0 0.032 0" rpy="1.5707963 0 0" />
+      <geometry><cylinder radius="0.058" length="0.03" /></geometry>
     </collision>
   </link>
@@ -225,20 +205,15 @@
       <geometry>
         <mesh
-          filename="package://chassis_description/meshes/w4.STL" />
-      </geometry>
-      <material
-        name="">
-        <color
-          rgba="1 1 1 1" />
-      </material>
-    </visual>
-    <collision>
-      <origin
-        xyz="0 0 0"
-        rpy="0 0 0" />
-      <geometry>
-        <mesh
-          filename="package://chassis_description/meshes/w4.STL" />
-      </geometry>
+          filename="package://chassis_description/meshes/decimated/w4.stl" />
+      </geometry>
+      <material
+        name="">
+        <color
+          rgba="1 1 1 1" />
+      </material>
+    </visual>
+    <collision>
+      <origin xyz="0 0.032 0" rpy="1.5707963 0 0" />
+      <geometry><cylinder radius="0.058" length="0.03" /></geometry>
     </collision>
   </link>

Commit message: feat(robot): 起伏底盘轮子 continuous + diff_drive（真轮驱动；加速度 1 m/s² 防翻），车体黄色/轮子深灰

File: src/rm_nav_bringup/urdf/sentry_robot_chassis_sim.xacro (robot description, xacro)
@@ -76,5 +76,5 @@
   <joint
     name="w1"
-    type="fixed">
+    type="continuous">
     <origin
       xyz="0.1615 -0.10895 -0.04"
@@ -85,5 +85,5 @@
       link="w1" />
     <axis
-      xyz="0 0 0" />
+      xyz="0 1 0" />
   </joint>
   <link
@@ -124,5 +124,5 @@
   <joint
     name="w2"
-    type="fixed">
+    type="continuous">
     <origin
       xyz="0.1615 0.17205 -0.04"
@@ -133,5 +133,5 @@
       link="w2" />
     <axis
-      xyz="0 0 0" />
+      xyz="0 1 0" />
   </joint>
   <link
@@ -172,5 +172,5 @@
   <joint
     name="w3"
-    type="fixed">
+    type="continuous">
     <origin
       xyz="-0.1615 -0.17205 -0.04"
@@ -181,5 +181,5 @@
       link="w3" />
     <axis
-      xyz="0 0 0" />
+      xyz="0 1 0" />
   </joint>
   <link
@@ -220,5 +220,5 @@
   <joint
     name="w4"
-    type="fixed">
+    type="continuous">
     <origin
       xyz="-0.1615 0.10895 -0.04"
@@ -229,5 +229,5 @@
       link="w4" />
     <axis
-      xyz="0 0 0" />
+      xyz="0 1 0" />
   </joint>
   <!-- 仿真附加（原 URDF 没有；几何/惯量/碰撞一律不动）-->
@@ -251,14 +251,27 @@
   </xacro:mid360>
   <gazebo>
-    <plugin name="mecanum_controller" filename="libgazebo_ros_planar_move.so">
+    <plugin name="diff_drive" filename="libgazebo_ros_diff_drive.so">
       <ros><namespace>/</namespace>
         <remapping>cmd_vel:=cmd_vel_chassis</remapping>
         <remapping>odom:=odom_ground_truth</remapping></ros>
-      <update_rate>100</update_rate><publish_rate>10</publish_rate>
-      <publish_odom>true</publish_odom><publish_odom_tf>false</publish_odom_tf>
-      <odometry_frame>odom</odometry_frame><robot_base_frame>base_link</robot_base_frame>
-      <covariance_x>0.0001</covariance_x><covariance_y>0.0001</covariance_y>
-      <covariance_yaw>0.01</covariance_yaw>
+      <update_rate>100</update_rate>
+      <left_joint>w1</left_joint>
+      <right_joint>w2</right_joint>
+      <wheel_separation>0.281</wheel_separation>
+      <wheel_diameter>0.116</wheel_diameter>
+      <max_wheel_torque>5.0</max_wheel_torque>
+      <max_wheel_acceleration>1.0</max_wheel_acceleration>
+      <command_topic>cmd_vel</command_topic>
+      <odometry_topic>odom</odometry_topic>
+      <odometry_frame>odom</odometry_frame>
+      <robot_base_frame>base_link</robot_base_frame>
+      <publish_odom>true</publish_odom>
+      <publish_odom_tf>false</publish_odom_tf>
     </plugin>
   </gazebo>
+  <gazebo reference="w1"><mu1>0.8</mu1><mu2>0.8</mu2><material>Gazebo/DarkGrey</material></gazebo>
+  <gazebo reference="w2"><mu1>0.8</mu1><mu2>0.8</mu2><material>Gazebo/DarkGrey</material></gazebo>
+  <gazebo reference="w3"><mu1>0.8</mu1><mu2>0.8</mu2><material>Gazebo/DarkGrey</material></gazebo>
+  <gazebo reference="w4"><mu1>0.8</mu1><mu2>0.8</mu2><material>Gazebo/DarkGrey</material></gazebo>
+  <gazebo reference="base_link"><material>Gazebo/Yellow</material></gazebo>
 </robot>

Commit message: fix(robot): 轮轴符号——左轮(w1,w3) +y、右轮(w2,w4) -y（差速驱动直行不原地转）

File: src/rm_nav_bringup/urdf/sentry_robot_chassis_sim.xacro (robot description, xacro)
@@ -84,6 +84,5 @@
     <child
       link="w1" />
-    <axis
-      xyz="0 1 0" />
+    <axis xyz="0 1 0" />
   </joint>
   <link
@@ -132,6 +131,5 @@
     <child
       link="w2" />
-    <axis
-      xyz="0 1 0" />
+    <axis xyz="0 -1 0" />
   </joint>
   <link
@@ -180,6 +178,5 @@
     <child
       link="w3" />
-    <axis
-      xyz="0 1 0" />
+    <axis xyz="0 1 0" />
   </joint>
   <link
@@ -228,6 +225,5 @@
     <child
       link="w4" />
-    <axis
-      xyz="0 1 0" />
+    <axis xyz="0 -1 0" />
   </joint>
   <!-- 仿真附加（原 URDF 没有；几何/惯量/碰撞一律不动）-->

Commit message: revert(robot): sim xacro 回到**纯原 URDF**（与 chassis.urdf 逐字节相同）+ 仅雷达/IMU/planar——让 Gazebo 与 RViz 的模型完全一致

File: src/rm_nav_bringup/urdf/sentry_robot_chassis_sim.xacro (robot description, xacro)
@@ -31,10 +31,15 @@
         name="">
         <color
-          rgba="1.0 0.85 0.1 1" />
-      </material>
-    </visual>
-    <collision>
-      <origin xyz="0 0 0.0295" rpy="0 0 0" />
-      <geometry><box size="0.456 0.446 0.097" /></geometry>
+          rgba="0.792156862745098 0.819607843137255 0.933333333333333 1" />
+      </material>
+    </visual>
+    <collision>
+      <origin
+        xyz="0 0 0"
+        rpy="0 0 0" />
+      <geometry>
+        <mesh
+          filename="package://chassis_description/meshes/base_link.STL" />
+      </geometry>
     </collision>
   </link>
@@ -66,17 +71,22 @@
         name="">
         <color
-          rgba="0.25 0.25 0.25 1" />
-      </material>
-    </visual>
-    <collision>
-      <origin xyz="0 -0.032 0" rpy="1.5707963 0 0" />
-      <geometry><cylinder radius="0.058" length="0.03" /></geometry>
+          rgba="1 1 1 1" />
+      </material>
+    </visual>
+    <collision>
+      <origin
+        xyz="0 0 0"
+        rpy="0 0 0" />
+      <geometry>
+        <mesh
+          filename="package://chassis_description/meshes/w1.STL" />
+      </geometry>
     </collision>
   </link>
   <joint
     name="w1"
-    type="continuous">
-    <origin
-      xyz="0.1615 -0.198 -0.04"
+    type="fixed">
+    <origin
+      xyz="0.1615 -0.10895 -0.04"
       rpy="0 0 0" />
     <parent
@@ -84,5 +94,6 @@
     <child
       link="w1" />
-    <axis xyz="0 1 0" />
+    <axis
+      xyz="0 0 0" />
   </joint>
   <link
@@ -113,17 +124,22 @@
         name="">
         <color
-          rgba="0.25 0.25 0.25 1" />
-      </material>
-    </visual>
-    <collision>
-      <origin xyz="0 -0.032 0" rpy="1.5707963 0 0" />
-      <geometry><cylinder radius="0.058" length="0.03" /></geometry>
+          rgba="1 1 1 1" />
+      </material>
+    </visual>
+    <collision>
+      <origin
+        xyz="0 0 0"
+        rpy="0 0 0" />
+      <geometry>
+        <mesh
+          filename="package://chassis_description/meshes/w2.STL" />
+      </geometry>
     </collision>
   </link>
   <joint
     name="w2"
-    type="continuous">
-    <origin
-      xyz="0.1615 0.262 -0.04"
+    type="fixed">
+    <origin
+      xyz="0.1615 0.17205 -0.04"
       rpy="0 0 0" />
     <parent
@@ -131,5 +147,6 @@
     <child
       link="w2" />
-    <axis xyz="0 -1 0" />
+    <axis
+      xyz="0 0 0" />
   </joint>
   <link
@@ -160,17 +177,22 @@
         name="">
         <color
-          rgba="0.25 0.25 0.25 1" />
-      </material>
-    </visual>
-    <collision>
-      <origin xyz="0 0.032 0" rpy="1.5707963 0 0" />
-      <geometry><cylinder radius="0.058" length="0.03" /></geometry>
+          rgba="1 1 1 1" />
+      </material>
+    </visual>
+    <collision>
+      <origin
+        xyz="0 0 0"
+        rpy="0 0 0" />
+      <geometry>
+        <mesh
+          filename="package://chassis_description/meshes/w3.STL" />
+      </geometry>
     </collision>
   </link>
   <joint
     name="w3"
-    type="continuous">
-    <origin
-      xyz="-0.1615 -0.262 -0.04"
+    type="fixed">
+    <origin
+      xyz="-0.1615 -0.17205 -0.04"
       rpy="0 0 0" />
     <parent
@@ -178,5 +200,6 @@
     <child
       link="w3" />
-    <axis xyz="0 1 0" />
+    <axis
+      xyz="0 0 0" />
   </joint>
   <link
@@ -207,17 +230,22 @@
         name="">
         <color
-          rgba="0.25 0.25 0.25 1" />
-      </material>
-    </visual>
-    <collision>
-      <origin xyz="0 0.032 0" rpy="1.5707963 0 0" />
-      <geometry><cylinder radius="0.058" length="0.03" /></geometry>
+          rgba="1 1 1 1" />
+      </material>
+    </visual>
+    <collision>
+      <origin
+        xyz="0 0 0"
+        rpy="0 0 0" />
+      <geometry>
+        <mesh
+          filename="package://chassis_description/meshes/w4.STL" />
+      </geometry>
     </collision>
   </link>
   <joint
     name="w4"
-    type="continuous">
-    <origin
-      xyz="-0.1615 0.198 -0.04"
+    type="fixed">
+    <origin
+      xyz="-0.1615 0.10895 -0.04"
       rpy="0 0 0" />
     <parent
@@ -225,7 +253,8 @@
     <child
       link="w4" />
-    <axis xyz="0 -1 0" />
-  </joint>
-  <!-- 仿真附加（原 URDF 没有；几何/惯量/碰撞一律不动）-->
+    <axis
+      xyz="0 0 0" />
+  </joint>
+  <!-- ===================== 仿真附加（原 URDF 没有；其余逐字节不动）===================== -->
   <link name="imu_link"/>
   <joint name="imu_joint" type="fixed">
@@ -247,27 +276,14 @@
   </xacro:mid360>
   <gazebo>
-    <plugin name="diff_drive" filename="libgazebo_ros_diff_drive.so">
+    <plugin name="mecanum_controller" filename="libgazebo_ros_planar_move.so">
       <ros><namespace>/</namespace>
         <remapping>cmd_vel:=cmd_vel_chassis</remapping>
         <remapping>odom:=odom_ground_truth</remapping></ros>
-      <update_rate>100</update_rate>
-      <left_joint>w1</left_joint>
-      <right_joint>w2</right_joint>
-      <wheel_separation>0.46</wheel_separation>
-      <wheel_diameter>0.116</wheel_diameter>
-      <max_wheel_torque>5.0</max_wheel_torque>
-      <max_wheel_acceleration>1.0</max_wheel_acceleration>
-      <command_topic>cmd_vel</command_topic>
-      <odometry_topic>odom</odometry_topic>
-      <odometry_frame>odom</odometry_frame>
-      <robot_base_frame>base_link</robot_base_frame>
-      <publish_odom>true</publish_odom>
-      <publish_odom_tf>false</publish_odom_tf>
+      <update_rate>100</update_rate><publish_rate>10</publish_rate>
+      <publish_odom>true</publish_odom><publish_odom_tf>false</publish_odom_tf>
+      <odometry_frame>odom</odometry_frame><robot_base_frame>base_link</robot_base_frame>
+      <covariance_x>0.0001</covariance_x><covariance_y>0.0001</covariance_y>
+      <covariance_yaw>0.01</covariance_yaw>
     </plugin>
   </gazebo>
-  <gazebo reference="w1"><mu1>0.8</mu1><mu2>0.8</mu2><material>Gazebo/DarkGrey</material></gazebo>
-  <gazebo reference="w2"><mu1>0.8</mu1><mu2>0.8</mu2><material>Gazebo/DarkGrey</material></gazebo>
-  <gazebo reference="w3"><mu1>0.8</mu1><mu2>0.8</mu2><material>Gazebo/DarkGrey</material></gazebo>
-  <gazebo reference="w4"><mu1>0.8</mu1><mu2>0.8</mu2><material>Gazebo/DarkGrey</material></gazebo>
-  <gazebo reference="base_link"><material>Gazebo/Yellow</material></gazebo>
 </robot>

Commit message: feat(robot): 起伏底盘质量对齐实车 ~10 kg（车体 9.2 + 4×0.2 轮；惯量按同比例缩放）

File: src/rm_nav_bringup/urdf/sentry_robot_chassis_sim.xacro (robot description, xacro)
@@ -11,12 +11,12 @@
         rpy="0 0 0" />
       <mass
-        value="4.30908483392141" />
-      <inertia
-        ixx="0.00356918503421658"
-        ixy="2.91111233555378E-06"
-        ixz="-1.58536389762567E-13"
-        iyy="0.00315932138586126"
-        iyz="-2.59640985562635E-14"
-        izz="0.00442129535026619" />
+        value="9.2" />
+      <inertia
+        ixx="0.007620296091"
+        ixy="6.215295e-06"
+        ixz="-0.0"
+        iyy="0.006745227321"
+        iyz="-0.0"
+        izz="0.009439572157" />
     </inertial>
     <visual>
@@ -51,12 +51,12 @@
         rpy="0 0 0" />
       <mass
-        value="0.0968885662811193" />
-      <inertia
-        ixx="0.000142054002080831"
-        ixy="-1.76056439722202E-16"
-        ixz="6.85752968055349E-16"
-        iyy="0.000270826964366967"
-        iyz="4.04461765349949E-17"
-        izz="0.000142054002078526" />
+        value="0.2" />
+      <inertia
+        ixx="0.000293231715"
+        ixy="-0.0"
+        ixz="0.0"
+        iyy="0.000559048348"
+        iyz="0.0"
+        izz="0.000293231715" />
     </inertial>
     <visual>
@@ -104,12 +104,12 @@
         rpy="0 0 0" />
       <mass
-        value="0.0968885662811196" />
-      <inertia
-        ixx="0.000142054002080838"
-        ixy="-1.7562802007376E-16"
-        ixz="6.85790224897307E-16"
-        iyy="0.000270826964366966"
-        iyz="4.0237417683157E-17"
-        izz="0.000142054002078533" />
+        value="0.2" />
+      <inertia
+        ixx="0.000293231715"
+        ixy="-0.0"
+        ixz="0.0"
+        iyy="0.000559048348"
+        iyz="0.0"
+        izz="0.000293231715" />
     </inertial>
     <visual>
@@ -157,12 +157,12 @@
         rpy="0 0 0" />
       <mass
-        value="0.096888566281119" />
-      <inertia
-        ixx="0.000142054002080834"
-        ixy="-1.75804051692341E-16"
-        ixz="-6.8568793984376E-16"
-        iyy="0.000270826964366966"
-        iyz="-4.0245017491951E-17"
-        izz="0.000142054002078529" />
+        value="0.2" />
+      <inertia
+        ixx="0.000293231715"
+        ixy="-0.0"
+        ixz="-0.0"
+        iyy="0.000559048348"
+        iyz="-0.0"
+        izz="0.000293231715" />
     </inertial>
     <visual>
@@ -210,12 +210,12 @@
         rpy="0 0 0" />
       <mass
-        value="0.0968885662811193" />
-      <inertia
-        ixx="0.000142054002080831"
-        ixy="-1.76056144471508E-16"
-        ixz="-6.85753899441331E-16"
-        iyy="0.000270826964366967"
-        iyz="-4.04759497027718E-17"
-        izz="0.000142054002078526" />
+        value="0.2" />
+      <inertia
+        ixx="0.000293231715"
+        ixy="-0.0"
+        ixz="-0.0"
+        iyy="0.000559048348"
+        iyz="-0.0"
+        izz="0.000293231715" />
     </inertial>
     <visual>

Commit message: style(robot): 车体黑色、轮子深灰（URDF 材质 + Gazebo 材质，RViz/Gazebo 一致）

File: src/rm_nav_bringup/urdf/sentry_robot_chassis_sim.xacro (robot description, xacro)
@@ -31,5 +31,5 @@
         name="">
         <color
-          rgba="0.792156862745098 0.819607843137255 0.933333333333333 1" />
+          rgba="0.02 0.02 0.02 1" />
       </material>
     </visual>
@@ -71,5 +71,5 @@
         name="">
         <color
-          rgba="1 1 1 1" />
+          rgba="0.22 0.22 0.22 1" />
       </material>
     </visual>
@@ -124,5 +124,5 @@
         name="">
         <color
-          rgba="1 1 1 1" />
+          rgba="0.22 0.22 0.22 1" />
       </material>
     </visual>
@@ -177,5 +177,5 @@
         name="">
         <color
-          rgba="1 1 1 1" />
+          rgba="0.22 0.22 0.22 1" />
       </material>
     </visual>
@@ -230,5 +230,5 @@
         name="">
         <color
-          rgba="1 1 1 1" />
+          rgba="0.22 0.22 0.22 1" />
       </material>
     </visual>
@@ -294,3 +294,9 @@
   <gazebo reference="w3"><mu1>0.02</mu1><mu2>0.02</mu2></gazebo>
   <gazebo reference="w4"><mu1>0.02</mu1><mu2>0.02</mu2></gazebo>
+  <!-- 颜色：车体黑、轮子深灰（Gazebo 渲染用；URDF 的 <visual> 材质给 RViz）-->
+  <gazebo reference="base_link"><material>Gazebo/Black</material></gazebo>
+  <gazebo reference="w1"><material>Gazebo/DarkGrey</material></gazebo>
+  <gazebo reference="w2"><material>Gazebo/DarkGrey</material></gazebo>
+  <gazebo reference="w3"><material>Gazebo/DarkGrey</material></gazebo>
+  <gazebo reference="w4"><material>Gazebo/DarkGrey</material></gazebo>
 </robot>

Commit message: feat(robot): 四轮真驱动——前/后各一个 diff_drive（w1/w2 + w3/w4 全驱动），连续轮+轴符号，μ0.8

File: src/rm_nav_bringup/urdf/sentry_robot_chassis_sim.xacro (robot description, xacro)
@@ -86,5 +86,5 @@
   <joint
     name="w1"
-    type="fixed">
+    type="continuous">
     <origin
       xyz="0.1615 -0.10895 -0.04"
@@ -94,6 +94,5 @@
     <child
       link="w1" />
-    <axis
-      xyz="0 0 0" />
+    <axis xyz="0 1 0" />
   </joint>
   <link
@@ -139,5 +138,5 @@
   <joint
     name="w2"
-    type="fixed">
+    type="continuous">
     <origin
       xyz="0.1615 0.17205 -0.04"
@@ -147,6 +146,5 @@
     <child
       link="w2" />
-    <axis
-      xyz="0 0 0" />
+    <axis xyz="0 -1 0" />
   </joint>
   <link
@@ -192,5 +190,5 @@
   <joint
     name="w3"
-    type="fixed">
+    type="continuous">
     <origin
       xyz="-0.1615 -0.17205 -0.04"
@@ -200,6 +198,5 @@
     <child
       link="w3" />
-    <axis
-      xyz="0 0 0" />
+    <axis xyz="0 1 0" />
   </joint>
   <link
@@ -245,5 +242,5 @@
   <joint
     name="w4"
-    type="fixed">
+    type="continuous">
     <origin
       xyz="-0.1615 0.10895 -0.04"
@@ -253,6 +250,5 @@
     <child
       link="w4" />
-    <axis
-      xyz="0 0 0" />
+    <axis xyz="0 -1 0" />
   </joint>
   <!-- ===================== 仿真附加（原 URDF 没有；其余逐字节不动）===================== -->
@@ -276,13 +272,40 @@
   </xacro:mid360>
   <gazebo>
-    <plugin name="mecanum_controller" filename="libgazebo_ros_planar_move.so">
+    <plugin name="diff_drive_front" filename="libgazebo_ros_diff_drive.so">
       <ros><namespace>/</namespace>
         <remapping>cmd_vel:=cmd_vel_chassis</remapping>
         <remapping>odom:=odom_ground_truth</remapping></ros>
-      <update_rate>100</update_rate><publish_rate>10</publish_rate>
-      <publish_odom>true</publish_odom><publish_odom_tf>false</publish_odom_tf>
-      <odometry_frame>odom</odometry_frame><robot_base_frame>base_link</robot_base_frame>
-      <covariance_x>0.0001</covariance_x><covariance_y>0.0001</covariance_y>
-      <covariance_yaw>0.01</covariance_yaw>
+      <update_rate>100</update_rate>
+      <left_joint>w1</left_joint>
+      <right_joint>w2</right_joint>
+      <wheel_separation>0.281</wheel_separation>
+      <wheel_diameter>0.116</wheel_diameter>
+      <max_wheel_torque>5.0</max_wheel_torque>
+      <max_wheel_acceleration>1.0</max_wheel_acceleration>
+      <command_topic>cmd_vel</command_topic>
+      <odometry_topic>odom</odometry_topic>
+      <odometry_frame>odom</odometry_frame>
+      <robot_base_frame>base_link</robot_base_frame>
+      <publish_odom>true</publish_odom>
+      <publish_odom_tf>false</publish_odom_tf>
+    </plugin>
+  </gazebo>
+  <gazebo>
+    <plugin name="diff_drive_rear" filename="libgazebo_ros_diff_drive.so">
+      <ros><namespace>/</namespace>
+        <remapping>cmd_vel:=cmd_vel_chassis</remapping></ros>
+      <update_rate>100</update_rate>
+      <left_joint>w3</left_joint>
+      <right_joint>w4</right_joint>
+      <wheel_separation>0.281</wheel_separation>
+      <wheel_diameter>0.116</wheel_diameter>
+      <max_wheel_torque>5.0</max_wheel_torque>
+      <max_wheel_acceleration>1.0</max_wheel_acceleration>
+      <command_topic>cmd_vel</command_topic>
+      <odometry_topic>odom</odometry_topic>
+      <odometry_frame>odom</odometry_frame>
+      <robot_base_frame>base_link</robot_base_frame>
+      <publish_odom>false</publish_odom>
+      <publish_odom_tf>false</publish_odom_tf>
     </plugin>
   </gazebo>
@@ -290,8 +313,8 @@
        默认 μ=1 时轮子"抓住"地面，planar_move 直接推底盘会在斜坡/台阶处产生倾覆力矩（翻车）；
        降到 μ=0.02 ⇒ 轮子滑动、底盘被速度直接推上去 ⇒ 不翻。只改摩擦，不改几何。 -->
-  <gazebo reference="w1"><mu1>0.02</mu1><mu2>0.02</mu2></gazebo>
-  <gazebo reference="w2"><mu1>0.02</mu1><mu2>0.02</mu2></gazebo>
-  <gazebo reference="w3"><mu1>0.02</mu1><mu2>0.02</mu2></gazebo>
-  <gazebo reference="w4"><mu1>0.02</mu1><mu2>0.02</mu2></gazebo>
+  <gazebo reference="w1"><mu1>0.8</mu1><mu2>0.8</mu2></gazebo>
+  <gazebo reference="w2"><mu1>0.8</mu1><mu2>0.8</mu2></gazebo>
+  <gazebo reference="w3"><mu1>0.8</mu1><mu2>0.8</mu2></gazebo>
+  <gazebo reference="w4"><mu1>0.8</mu1><mu2>0.8</mu2></gazebo>
   <!-- 颜色：车体黑、轮子深灰（Gazebo 渲染用；URDF 的 <visual> 材质给 RViz）-->
   <gazebo reference="base_link"><material>Gazebo/Black</material></gazebo>
