Commit message: revert(robot): sim xacro 回到开始那版（00cd9f9：纯原模型 + 平放雷达/IMU + planar_move；轮子固定）

File: src/rm_nav_bringup/urdf/sentry_robot_chassis_sim.xacro (robot description, xacro)
@@ -11,12 +11,12 @@
         rpy="0 0 0" />
       <mass
-        value="9.2" />
-      <inertia
-        ixx="0.007620296091"
-        ixy="6.215295e-06"
-        ixz="-0.0"
-        iyy="0.006745227321"
-        iyz="-0.0"
-        izz="0.009439572157" />
+        value="4.30908483392141" />
+      <inertia
+        ixx="0.00356918503421658"
+        ixy="2.91111233555378E-06"
+        ixz="-1.58536389762567E-13"
+        iyy="0.00315932138586126"
+        iyz="-2.59640985562635E-14"
+        izz="0.00442129535026619" />
     </inertial>
     <visual>
@@ -31,15 +31,10 @@
         name="">
         <color
-          rgba="0.02 0.02 0.02 1" />
-      </material>
-    </visual>
-    <collision>
-      <origin
-        xyz="0 0 0"
-        rpy="0 0 0" />
-      <geometry>
-        <mesh
-          filename="package://chassis_description/meshes/base_link.STL" />
-      </geometry>
+          rgba="0.792156862745098 0.819607843137255 0.933333333333333 1" />
+      </material>
+    </visual>
+    <collision>
+      <origin xyz="0 0 0.0295" rpy="0 0 0" />
+      <geometry><box size="0.456 0.446 0.097" /></geometry>
     </collision>
   </link>
@@ -51,12 +46,12 @@
         rpy="0 0 0" />
       <mass
-        value="0.2" />
-      <inertia
-        ixx="0.000293231715"
-        ixy="-0.0"
-        ixz="0.0"
-        iyy="0.000559048348"
-        iyz="0.0"
-        izz="0.000293231715" />
+        value="0.0968885662811193" />
+      <inertia
+        ixx="0.000142054002080831"
+        ixy="-1.76056439722202E-16"
+        ixz="6.85752968055349E-16"
+        iyy="0.000270826964366967"
+        iyz="4.04461765349949E-17"
+        izz="0.000142054002078526" />
     </inertial>
     <visual>
@@ -71,20 +66,15 @@
         name="">
         <color
-          rgba="0.22 0.22 0.22 1" />
-      </material>
-    </visual>
-    <collision>
-      <origin
-        xyz="0 0 0"
-        rpy="0 0 0" />
-      <geometry>
-        <mesh
-          filename="package://chassis_description/meshes/w1.STL" />
-      </geometry>
+          rgba="1 1 1 1" />
+      </material>
+    </visual>
+    <collision>
+      <origin xyz="0 -0.032 0" rpy="1.5707963 0 0" />
+      <geometry><cylinder radius="0.058" length="0.03" /></geometry>
     </collision>
   </link>
   <joint
     name="w1"
-    type="continuous">
+    type="fixed">
     <origin
       xyz="0.1615 -0.10895 -0.04"
@@ -94,5 +84,6 @@
     <child
       link="w1" />
-    <axis xyz="0 1 0" />
+    <axis
+      xyz="0 0 0" />
   </joint>
   <link
@@ -103,12 +94,12 @@
         rpy="0 0 0" />
       <mass
-        value="0.2" />
-      <inertia
-        ixx="0.000293231715"
-        ixy="-0.0"
-        ixz="0.0"
-        iyy="0.000559048348"
-        iyz="0.0"
-        izz="0.000293231715" />
+        value="0.0968885662811196" />
+      <inertia
+        ixx="0.000142054002080838"
+        ixy="-1.7562802007376E-16"
+        ixz="6.85790224897307E-16"
+        iyy="0.000270826964366966"
+        iyz="4.0237417683157E-17"
+        izz="0.000142054002078533" />
     </inertial>
     <visual>
@@ -123,20 +114,15 @@
         name="">
         <color
-          rgba="0.22 0.22 0.22 1" />
-      </material>
-    </visual>
-    <collision>
-      <origin
-        xyz="0 0 0"
-        rpy="0 0 0" />
-      <geometry>
-        <mesh
-          filename="package://chassis_description/meshes/w2.STL" />
-      </geometry>
+          rgba="1 1 1 1" />
+      </material>
+    </visual>
+    <collision>
+      <origin xyz="0 -0.032 0" rpy="1.5707963 0 0" />
+      <geometry><cylinder radius="0.058" length="0.03" /></geometry>
     </collision>
   </link>
   <joint
     name="w2"
-    type="continuous">
+    type="fixed">
     <origin
       xyz="0.1615 0.17205 -0.04"
@@ -146,5 +132,6 @@
     <child
       link="w2" />
-    <axis xyz="0 -1 0" />
+    <axis
+      xyz="0 0 0" />
   </joint>
   <link
@@ -155,12 +142,12 @@
         rpy="0 0 0" />
       <mass
-        value="0.2" />
-      <inertia
-        ixx="0.000293231715"
-        ixy="-0.0"
-        ixz="-0.0"
-        iyy="0.000559048348"
-        iyz="-0.0"
-        izz="0.000293231715" />
+        value="0.096888566281119" />
+      <inertia
+        ixx="0.000142054002080834"
+        ixy="-1.75804051692341E-16"
+        ixz="-6.8568793984376E-16"
+        iyy="0.000270826964366966"
+        iyz="-4.0245017491951E-17"
+        izz="0.000142054002078529" />
     </inertial>
     <visual>
@@ -175,20 +162,15 @@
         name="">
         <color
-          rgba="0.22 0.22 0.22 1" />
-      </material>
-    </visual>
-    <collision>
-      <origin
-        xyz="0 0 0"
-        rpy="0 0 0" />
-      <geometry>
-        <mesh
-          filename="package://chassis_description/meshes/w3.STL" />
-      </geometry>
+          rgba="1 1 1 1" />
+      </material>
+    </visual>
+    <collision>
+      <origin xyz="0 0.032 0" rpy="1.5707963 0 0" />
+      <geometry><cylinder radius="0.058" length="0.03" /></geometry>
     </collision>
   </link>
   <joint
     name="w3"
-    type="continuous">
+    type="fixed">
     <origin
       xyz="-0.1615 -0.17205 -0.04"
@@ -198,5 +180,6 @@
     <child
       link="w3" />
-    <axis xyz="0 1 0" />
+    <axis
+      xyz="0 0 0" />
   </joint>
   <link
@@ -207,12 +190,12 @@
         rpy="0 0 0" />
       <mass
-        value="0.2" />
-      <inertia
-        ixx="0.000293231715"
-        ixy="-0.0"
-        ixz="-0.0"
-        iyy="0.000559048348"
-        iyz="-0.0"
-        izz="0.000293231715" />
+        value="0.0968885662811193" />
+      <inertia
+        ixx="0.000142054002080831"
+        ixy="-1.76056144471508E-16"
+        ixz="-6.85753899441331E-16"
+        iyy="0.000270826964366967"
+        iyz="-4.04759497027718E-17"
+        izz="0.000142054002078526" />
     </inertial>
     <visual>
@@ -227,20 +210,15 @@
         name="">
         <color
-          rgba="0.22 0.22 0.22 1" />
-      </material>
-    </visual>
-    <collision>
-      <origin
-        xyz="0 0 0"
-        rpy="0 0 0" />
-      <geometry>
-        <mesh
-          filename="package://chassis_description/meshes/w4.STL" />
-      </geometry>
+          rgba="1 1 1 1" />
+      </material>
+    </visual>
+    <collision>
+      <origin xyz="0 0.032 0" rpy="1.5707963 0 0" />
+      <geometry><cylinder radius="0.058" length="0.03" /></geometry>
     </collision>
   </link>
   <joint
     name="w4"
-    type="continuous">
+    type="fixed">
     <origin
       xyz="-0.1615 0.10895 -0.04"
@@ -250,7 +228,8 @@
     <child
       link="w4" />
-    <axis xyz="0 -1 0" />
-  </joint>
-  <!-- ===================== 仿真附加（原 URDF 没有；其余逐字节不动）===================== -->
+    <axis
+      xyz="0 0 0" />
+  </joint>
+  <!-- 仿真附加（原 URDF 没有；几何/惯量/碰撞一律不动）-->
   <link name="imu_link"/>
   <joint name="imu_joint" type="fixed">
@@ -272,54 +251,14 @@
   </xacro:mid360>
   <gazebo>
-    <plugin name="diff_drive_front" filename="libgazebo_ros_diff_drive.so">
+    <plugin name="mecanum_controller" filename="libgazebo_ros_planar_move.so">
       <ros><namespace>/</namespace>
         <remapping>cmd_vel:=cmd_vel_chassis</remapping>
         <remapping>odom:=odom_ground_truth</remapping></ros>
-      <update_rate>100</update_rate>
-      <left_joint>w1</left_joint>
-      <right_joint>w2</right_joint>
-      <wheel_separation>0.281</wheel_separation>
-      <wheel_diameter>0.116</wheel_diameter>
-      <max_wheel_torque>5.0</max_wheel_torque>
-      <max_wheel_acceleration>1.0</max_wheel_acceleration>
-      <command_topic>cmd_vel</command_topic>
-      <odometry_topic>odom</odometry_topic>
-      <odometry_frame>odom</odometry_frame>
-      <robot_base_frame>base_link</robot_base_frame>
-      <publish_odom>true</publish_odom>
-      <publish_odom_tf>false</publish_odom_tf>
+      <update_rate>100</update_rate><publish_rate>10</publish_rate>
+      <publish_odom>true</publish_odom><publish_odom_tf>false</publish_odom_tf>
+      <odometry_frame>odom</odometry_frame><robot_base_frame>base_link</robot_base_frame>
+      <covariance_x>0.0001</covariance_x><covariance_y>0.0001</covariance_y>
+      <covariance_yaw>0.01</covariance_yaw>
     </plugin>
   </gazebo>
-  <gazebo>
-    <plugin name="diff_drive_rear" filename="libgazebo_ros_diff_drive.so">
-      <ros><namespace>/</namespace>
-        <remapping>cmd_vel:=cmd_vel_chassis</remapping></ros>
-      <update_rate>100</update_rate>
-      <left_joint>w3</left_joint>
-      <right_joint>w4</right_joint>
-      <wheel_separation>0.281</wheel_separation>
-      <wheel_diameter>0.116</wheel_diameter>
-      <max_wheel_torque>5.0</max_wheel_torque>
-      <max_wheel_acceleration>1.0</max_wheel_acceleration>
-      <command_topic>cmd_vel</command_topic>
-      <odometry_topic>odom</odometry_topic>
-      <odometry_frame>odom</odometry_frame>
-      <robot_base_frame>base_link</robot_base_frame>
-      <publish_odom>false</publish_odom>
-      <publish_odom_tf>false</publish_odom_tf>
-    </plugin>
-  </gazebo>
-  <!-- 轮子对地摩擦：与 robot11 同款（固定轮 + planar_move 的组合）——
-       默认 μ=1 时轮子"抓住"地面，planar_move 直接推底盘会在斜坡/台阶处产生倾覆力矩（翻车）；
-       降到 μ=0.02 ⇒ 轮子滑动、底盘被速度直接推上去 ⇒ 不翻。只改摩擦，不改几何。 -->
-  <gazebo reference="w1"><mu1>0.8</mu1><mu2>0.8</mu2></gazebo>
-  <gazebo reference="w2"><mu1>0.8</mu1><mu2>0.8</mu2></gazebo>
-  <gazebo reference="w3"><mu1>0.8</mu1><mu2>0.8</mu2></gazebo>
-  <gazebo reference="w4"><mu1>0.8</mu1><mu2>0.8</mu2></gazebo>
-  <!-- 颜色：车体黑、轮子深灰（Gazebo 渲染用；URDF 的 <visual> 材质给 RViz）-->
-  <gazebo reference="base_link"><material>Gazebo/Black</material></gazebo>
-  <gazebo reference="w1"><material>Gazebo/DarkGrey</material></gazebo>
-  <gazebo reference="w2"><material>Gazebo/DarkGrey</material></gazebo>
-  <gazebo reference="w3"><material>Gazebo/DarkGrey</material></gazebo>
-  <gazebo reference="w4"><material>Gazebo/DarkGrey</material></gazebo>
 </robot>

Commit message: style(robot): 车体黑色（URDF + Gazebo 材质），轮子深灰

File: src/rm_nav_bringup/urdf/sentry_robot_chassis_sim.xacro (robot description, xacro)
@@ -31,5 +31,5 @@
         name="">
         <color
-          rgba="0.792156862745098 0.819607843137255 0.933333333333333 1" />
+          rgba="0.02 0.02 0.02 1" />
       </material>
     </visual>
@@ -66,5 +66,5 @@
         name="">
         <color
-          rgba="1 1 1 1" />
+          rgba="0.22 0.22 0.22 1" />
       </material>
     </visual>
@@ -114,5 +114,5 @@
         name="">
         <color
-          rgba="1 1 1 1" />
+          rgba="0.22 0.22 0.22 1" />
       </material>
     </visual>
@@ -162,5 +162,5 @@
         name="">
         <color
-          rgba="1 1 1 1" />
+          rgba="0.22 0.22 0.22 1" />
       </material>
     </visual>
@@ -210,5 +210,5 @@
         name="">
         <color
-          rgba="1 1 1 1" />
+          rgba="0.22 0.22 0.22 1" />
       </material>
     </visual>
@@ -262,3 +262,8 @@
     </plugin>
   </gazebo>
+  <gazebo reference="base_link"><material>Gazebo/Black</material></gazebo>
+  <gazebo reference="w1"><material>Gazebo/DarkGrey</material></gazebo>
+  <gazebo reference="w2"><material>Gazebo/DarkGrey</material></gazebo>
+  <gazebo reference="w3"><material>Gazebo/DarkGrey</material></gazebo>
+  <gazebo reference="w4"><material>Gazebo/DarkGrey</material></gazebo>
 </robot>

Commit message: feat(robot): 雷达物理倾斜 45° 下俯（livox_physical 挂传感器 + livox_frame 水平数据帧，extrinsic 旋正）

File: src/rm_nav_bringup/urdf/sentry_robot_chassis_sim.xacro (robot description, xacro)
@@ -247,7 +247,19 @@
   </gazebo>
   <xacro:include filename="$(find ros2_livox_simulation)/urdf/mid360.xacro"/>
-  <xacro:mid360 name="livox_frame" parent="base_link" topic="/livox/lidar">
+  <!-- ★ 2026-10-30：雷达**物理倾斜 45° 下俯**（与实车一致）——与 robot11 同款"物理/数据两层"：
+       ① livox_physical：物理安装位置（rpy=-45° 下俯），**射线传感器挂这里** ⇒ 插件发
+          /livox/lidar_raw（点表达在**斜的**物理系）；
+       ② livox_frame：**水平的数据帧**（rpy=0），只做 TF 锚点；
+       ③ launch 里的 livox_cloud_extrinsic 用 TF(livox_frame←livox_physical) 把点云旋正 →
+          /livox/lidar（frame_id=livox_frame）⇒ 下游（linefit/patchwork/LIO）看到的仍是水平点云。 -->
+  <xacro:mid360 name="livox_physical" parent="base_link" topic="/livox/lidar_raw">
+    <origin xyz="0 0 0.09" rpy="-0.78539816 0 0"/>
+  </xacro:mid360>
+  <!-- 水平数据帧（与物理雷达同位置，rpy=0；无 visual）-->
+  <link name="livox_frame"/>
+  <joint name="livox_frame_joint" type="fixed">
     <origin xyz="0 0 0.09" rpy="0 0 0"/>
-  </xacro:mid360>
+    <parent link="base_link"/><child link="livox_frame"/>
+  </joint>
   <gazebo>
     <plugin name="mecanum_controller" filename="libgazebo_ros_planar_move.so">

Commit message: tune(robot): 雷达下俯 45° -> 30°（与 robot11 一致，FOV 能看墙/远处；物理/数据两层不变）

File: src/rm_nav_bringup/urdf/sentry_robot_chassis_sim.xacro (robot description, xacro)
@@ -254,5 +254,5 @@
           /livox/lidar（frame_id=livox_frame）⇒ 下游（linefit/patchwork/LIO）看到的仍是水平点云。 -->
   <xacro:mid360 name="livox_physical" parent="base_link" topic="/livox/lidar_raw">
-    <origin xyz="0 0 0.09" rpy="-0.78539816 0 0"/>
+    <origin xyz="0 0 0.09" rpy="-0.52359878 0 0"/>
   </xacro:mid360>
   <!-- 水平数据帧（与物理雷达同位置，rpy=0；无 visual）-->

Commit message: revert(robot): mecanum 试用遇到 gazebo_ros2_control 的 robot_description 参数解析问题 —— 先恢复 planar 可用状态；mecanum_controller.yaml 保留供后续继续

File: src/rm_nav_bringup/urdf/sentry_robot_chassis_sim.xacro (robot description, xacro)
@@ -247,19 +247,7 @@
   </gazebo>
   <xacro:include filename="$(find ros2_livox_simulation)/urdf/mid360.xacro"/>
-  <!-- ★ 2026-10-30：雷达**物理倾斜 45° 下俯**（与实车一致）——与 robot11 同款"物理/数据两层"：
-       ① livox_physical：物理安装位置（rpy=-30° 下俯），**射线传感器挂这里** ⇒ 插件发
-          /livox/lidar_raw（点表达在**斜的**物理系）；
-       ② livox_frame：**水平的数据帧**（rpy=0），只做 TF 锚点；
-       ③ launch 里的 livox_cloud_extrinsic 用 TF(livox_frame←livox_physical) 把点云旋正 →
-          /livox/lidar（frame_id=livox_frame）⇒ 下游（linefit/patchwork/LIO）看到的仍是水平点云。 -->
-  <xacro:mid360 name="livox_physical" parent="base_link" topic="/livox/lidar_raw">
-    <origin xyz="0 0 0.09" rpy="-0.52359878 0 0"/>
+  <xacro:mid360 name="livox_frame" parent="base_link" topic="/livox/lidar">
+    <origin xyz="0 0 0.09" rpy="0 0 0"/>
   </xacro:mid360>
-  <!-- 水平数据帧（与物理雷达同位置，rpy=0；无 visual）-->
-  <link name="livox_frame"/>
-  <joint name="livox_frame_joint" type="fixed">
-    <origin xyz="0 0 0.09" rpy="0 0 0"/>
-    <parent link="base_link"/><child link="livox_frame"/>
-  </joint>
   <gazebo>
     <plugin name="mecanum_controller" filename="libgazebo_ros_planar_move.so">
@@ -279,9 +267,3 @@
   <gazebo reference="w3"><material>Gazebo/DarkGrey</material></gazebo>
   <gazebo reference="w4"><material>Gazebo/DarkGrey</material></gazebo>
-  <!-- 轮子对地摩擦 0.02（robot11 同款）：固定轮+planar_move 时，默认 μ=1 会让轮子"抓地"
-       而在加速/急转/坡道产生倾覆力矩（翻车）；0.02 让轮子滑动、底盘被速度直接推 ⇒ 不翻。 -->
-  <gazebo reference="w1"><mu1>0.02</mu1><mu2>0.02</mu2></gazebo>
-  <gazebo reference="w2"><mu1>0.02</mu1><mu2>0.02</mu2></gazebo>
-  <gazebo reference="w3"><mu1>0.02</mu1><mu2>0.02</mu2></gazebo>
-  <gazebo reference="w4"><mu1>0.02</mu1><mu2>0.02</mu2></gazebo>
 </robot>

Commit message: feat(robot): 自定义麦轮驱动插件（cw 直行验证通过；4 轮 joint 改名避免 link 撞名；插件自发布 /joint_states 与 /odom_ground_truth）

File: src/rm_nav_bringup/urdf/sentry_robot_chassis_sim.xacro (robot description, xacro)
@@ -75,6 +75,6 @@
   </link>
   <joint
-    name="w1"
-    type="fixed">
+    name="w1_joint"
+    type="continuous">
     <origin
       xyz="0.1615 -0.10895 -0.04"
@@ -84,6 +84,5 @@
     <child
       link="w1" />
-    <axis
-      xyz="0 0 0" />
+    <axis xyz="0 1 0" />
   </joint>
   <link
@@ -123,6 +122,6 @@
   </link>
   <joint
-    name="w2"
-    type="fixed">
+    name="w2_joint"
+    type="continuous">
     <origin
       xyz="0.1615 0.17205 -0.04"
@@ -132,6 +131,5 @@
     <child
       link="w2" />
-    <axis
-      xyz="0 0 0" />
+    <axis xyz="0 1 0" />
   </joint>
   <link
@@ -171,6 +169,6 @@
   </link>
   <joint
-    name="w3"
-    type="fixed">
+    name="w3_joint"
+    type="continuous">
     <origin
       xyz="-0.1615 -0.17205 -0.04"
@@ -180,6 +178,5 @@
     <child
       link="w3" />
-    <axis
-      xyz="0 0 0" />
+    <axis xyz="0 1 0" />
   </joint>
   <link
@@ -219,6 +216,6 @@
   </link>
   <joint
-    name="w4"
-    type="fixed">
+    name="w4_joint"
+    type="continuous">
     <origin
       xyz="-0.1615 0.10895 -0.04"
@@ -228,6 +225,5 @@
     <child
       link="w4" />
-    <axis
-      xyz="0 0 0" />
+    <axis xyz="0 1 0" />
   </joint>
   <!-- 仿真附加（原 URDF 没有；几何/惯量/碰撞一律不动）-->
@@ -250,14 +246,13 @@
     <origin xyz="0 0 0.09" rpy="0 0 0"/>
   </xacro:mid360>
+  <!-- ★ 2026-10-31：自定义麦轮驱动插件（绕开 gazebo_ros2_control 的 robot_description 解析坑）
+       /cmd_vel_chassis (vx,vy,wz) → 4 轮速度（麦轮逆解）→ 轮子真滚；
+       /odom_ground_truth 发模型世界位姿。 -->
   <gazebo>
-    <plugin name="mecanum_controller" filename="libgazebo_ros_planar_move.so">
-      <ros><namespace>/</namespace>
-        <remapping>cmd_vel:=cmd_vel_chassis</remapping>
-        <remapping>odom:=odom_ground_truth</remapping></ros>
-      <update_rate>100</update_rate><publish_rate>10</publish_rate>
-      <publish_odom>true</publish_odom><publish_odom_tf>false</publish_odom_tf>
-      <odometry_frame>odom</odometry_frame><robot_base_frame>base_link</robot_base_frame>
-      <covariance_x>0.0001</covariance_x><covariance_y>0.0001</covariance_y>
-      <covariance_yaw>0.01</covariance_yaw>
+    <plugin name="mecanum_drive" filename="libchassis_mecanum_drive.so">
+      <wheel_radius>0.058</wheel_radius>
+      <wheel_separation_sum>0.302</wheel_separation_sum>
+      <cmd_timeout>0.5</cmd_timeout>
+      <max_wheel_speed>40.0</max_wheel_speed>
     </plugin>
   </gazebo>

Commit message: fix(chassis drive): 运动学驱动 + yaw 标定 —— 前进/左转/右转方向与速度都对（实测 0.201 m/s、±0.46 rad/s）；去掉 joint_states 发布（清掉 TF_OLD_DATA 刷屏）

File: src/rm_nav_bringup/urdf/sentry_robot_chassis_sim.xacro (robot description, xacro)
@@ -85,4 +85,6 @@
       link="w1" />
     <axis xyz="0 1 0" />
+    <limit effort="20.0" velocity="60.0" />
+    <dynamics damping="0.02" friction="0.0" />
   </joint>
   <link
@@ -132,4 +134,6 @@
       link="w2" />
     <axis xyz="0 1 0" />
+    <limit effort="20.0" velocity="60.0" />
+    <dynamics damping="0.02" friction="0.0" />
   </joint>
   <link
@@ -179,4 +183,6 @@
       link="w3" />
     <axis xyz="0 1 0" />
+    <limit effort="20.0" velocity="60.0" />
+    <dynamics damping="0.02" friction="0.0" />
   </joint>
   <link
@@ -226,4 +232,6 @@
       link="w4" />
     <axis xyz="0 1 0" />
+    <limit effort="20.0" velocity="60.0" />
+    <dynamics damping="0.02" friction="0.0" />
   </joint>
   <!-- 仿真附加（原 URDF 没有；几何/惯量/碰撞一律不动）-->
@@ -255,10 +263,27 @@
       <cmd_timeout>0.5</cmd_timeout>
       <max_wheel_speed>40.0</max_wheel_speed>
+      <yaw_gain>5.0</yaw_gain>
     </plugin>
   </gazebo>
   <gazebo reference="base_link"><material>Gazebo/Black</material></gazebo>
-  <gazebo reference="w1"><material>Gazebo/DarkGrey</material></gazebo>
-  <gazebo reference="w2"><material>Gazebo/DarkGrey</material></gazebo>
-  <gazebo reference="w3"><material>Gazebo/DarkGrey</material></gazebo>
-  <gazebo reference="w4"><material>Gazebo/DarkGrey</material></gazebo>
+  <gazebo reference="w1">
+    <material>Gazebo/DarkGrey</material>
+    <mu1>1.0</mu1><mu2>0.01</mu2>
+    <fdir1>1 0 0</fdir1>
+  </gazebo>
+  <gazebo reference="w2">
+    <material>Gazebo/DarkGrey</material>
+    <mu1>1.0</mu1><mu2>0.01</mu2>
+    <fdir1>1 0 0</fdir1>
+  </gazebo>
+  <gazebo reference="w3">
+    <material>Gazebo/DarkGrey</material>
+    <mu1>1.0</mu1><mu2>0.01</mu2>
+    <fdir1>1 0 0</fdir1>
+  </gazebo>
+  <gazebo reference="w4">
+    <material>Gazebo/DarkGrey</material>
+    <mu1>1.0</mu1><mu2>0.01</mu2>
+    <fdir1>1 0 0</fdir1>
+  </gazebo>
 </robot>
